Commit message: update every sensor macro to the geometry inserter macro

File: defs/sensors/imaging/camera.xacro (robot description, xacro)
@@ -4,85 +4,74 @@
        xmlns:interface="http://playerstage.sourceforge.net/gazebo/xmlschema/#interface"
        xmlns:xacro="http://ros.org/wiki/xacro">
-<xacro:include filename="$(find rapid_robot_xacros)/defs/constants.xacro"/>
+<xacro:include filename="$(find rapid_robot_xacros)/defs/geometry/geo_ins.xacro"/>
 <!-- Example -->
 <!--
 <xacro:rr_cam
-		name             ="cam0"
-	 	robot_namespace  ="${robot_namespace}"
-		parent_link      ="chassis"
-		x                ="${chassis_len/2}"
-	    y                ="0"
-        z                ="0"
-        roll             ="0"
-        pitch            ="-0.01"
-        yaw              ="0"
-		always_on        ="true"
-		frame_name       ="camera0"
-		image_width      ="640"
-		image_height     ="480"
-		image_format     ="R8G8B8"
-		clip_near        ="0.02"
-		clip_far         ="300"
-		noise_type       ="gaussian"
-		noise_mean       ="0.0"
-		noise_std_dev    ="0.007"
-		fov              ="0.873"
-		hack_baseline    ="0.07"
-		dist_K1          ="0.0"
-		dist_K2          ="0.0"
-		dist_K3          ="0.0"
-		dist_T1          ="0.0"
-		dist_T2          ="0.0"
-		update_rate      ="30"
-        />
+	name             ="cam0"
+ 	robot_namespace  ="${robot_namespace}"
+	always_on        ="true"
+	frame_name       ="camera0"
+	image_width      ="640"
+	image_height     ="480"
+	image_format     ="R8G8B8"
+	clip_near        ="0.02"
+	clip_far         ="300"
+	noise_type       ="gaussian"
+	noise_mean       ="0.0"
+	noise_std_dev    ="0.007"
+	fov              ="0.873"
+	hack_baseline    ="0.07"
+	dist_K1          ="0.0"
+	dist_K2          ="0.0"
+	dist_K3          ="0.0"
+	dist_T1          ="0.0"
+	dist_T2          ="0.0"
+	update_rate      ="30"
+	parent           ="base_link"
+    has_inertia      ="false"
+	>
+	<origin xyz="${chassis_len/2}
+                 0
+	             ${chassis_center}" rpy="0 0 0" />
+	<geometry>
+		<box size="0.02 0.02 0.02" />
+	</geometry>
+	<material name="Yellow">
+		<color rgba="0 0 0 1"/>
+	</material>
+	 <inertial/>
+    </xacro:rr_cam>
+	<xacro:rr_gaz_mat_s name="cam0" material="Gazebo/FlatBlack"/>
 -->
-<xacro:macro name="rr_cam" params="
-	 							name
-	 							robot_namespace
-								parent_link
-								x y z roll pitch yaw
-								always_on
-								frame_name
-								image_width
-								image_height
-								image_format
-								clip_near
-								clip_far
-								noise_type
-								noise_mean
-								noise_std_dev
-								fov
-								hack_baseline
-								dist_K1
-								dist_K2
-								dist_K3
-								dist_T1
-								dist_T2
-								update_rate
-	                            ">
-<link name="${name}_link">
-	<visual>
-		<origin xyz="0 0 0"
-		        rpy="0 0 0"/>
-		<geometry>
-			<box size="0.02 0.02 0.02" />
-		</geometry>
-		<material name="Black">
-			<color rgba="0.0 0.0 0.0 1.0"/>
-		</material>
-	</visual>
-	<collision>
-		<origin xyz="0 0 0"
-		        rpy="0 0 0"/>
-		<geometry>
-			<box size="0.02 0.02 0.02" />
-		</geometry>
-	</collision>
-</link>
-<joint name="${name}_joint" type="fixed">
-	<origin xyz="${x} ${y} ${z}" rpy="${roll} ${pitch} ${yaw}"/>
-	<parent link="${parent_link}"/>
-	<child link="${name}_link"/>
-</joint>
+<xacro:macro name="rr_cam"
+	params="
+			name
+			robot_namespace
+			always_on
+			frame_name
+			image_width
+			image_height
+			image_format
+			clip_near
+			clip_far
+			noise_type
+			noise_mean
+			noise_std_dev
+			fov
+			hack_baseline
+			dist_K1
+			dist_K2
+			dist_K3
+			dist_T1
+			dist_T2
+			update_rate
+			parent
+	        has_inertia
+		    *origin
+		    *geometry
+		    *material
+		    *inertial
+	        ">
+<xacro:rr_geo_ins/>
 <gazebo reference="${name}_link">
 	<material value="Gazebo/FlatBlack" />

File: defs/sensors/inertia/imu.xacro (robot description, xacro)
@@ -5,11 +5,37 @@
        xmlns:xacro="http://ros.org/wiki/xacro"
 >
+<xacro:include filename="$(find rapid_robot_xacros)/defs/geometry/geo_ins.xacro"/>
 <!-- Example -->
 <!--
+<xacro:rr_imu
+	name="imu0"
+ 	robot_namespace=""
+	topic_name="/imu"
+	gaussian_noise="2.89e-08"
+	imu_x="0"
+	imu_y="0"
+	imu_z="0"
+	imu_roll="0"
+	imu_pitch="0"
+	imu_yaw="0"
+	parent="base_link"
+	has_inertia="false"
+	>
+	<origin xyz="${wheel_base_center_x}
+                   0
+	             ${chassis_center-((chassis_floor_clearance+
+                   chassis_height/2)-(wheel_diameter/2))}" rpy="0 0 0" />
+	<geometry>
+		<box size="0.02 0.02 0.02" />
+	</geometry>
+	<material name="Yellow">
+		<color rgba="1 1 0 1"/>
+	</material>
+	 <inertial/>
+</xacro:rr_imu>
 -->
 <xacro:macro name="rr_imu" params="name
 								robot_namespace
 								topic_name
-								parent_link
 								gaussian_noise
 								imu_x
@@ -19,4 +45,5 @@
 								imu_pitch
 								imu_yaw
+								parent
 	                            has_inertia
 							    *origin
@@ -25,21 +52,5 @@
 							    *inertial
 								">
-<link name="${name}_link">
-  <visual>
-      <xacro:insert_block name="geometry" />
-	  <xacro:insert_block name="material" />
-  </visual>
-  <collision name="${name}_collision">
-  	  	<xacro:insert_block name="geometry" />
-  </collision>
-  <xacro:if value="${has_inertia}">
-	<xacro:insert_block name="inertial" />
-  </xacro:if>
-</link>
-<joint name="${name}_joint" type="fixed">
-	<parent link="${parent_link}" />
-	<child link="${name}_link" />
-	<xacro:insert_block name="origin" />
-</joint>
+<xacro:rr_geo_ins/>
 <gazebo>
 	  <plugin name="imu{id}_controller" filename="libgazebo_ros_imu.so">

File: defs/sensors/position/gps.xacro (robot description, xacro)
@@ -5,4 +5,5 @@
        xmlns:xacro="http://ros.org/wiki/xacro"
 >
+<xacro:include filename="$(find rapid_robot_xacros)/defs/geometry/geo_ins.xacro"/>
 <!-- Example -->
 <!--
@@ -10,5 +11,4 @@
 		name="gps0"
 	 	robot_namespace="${robot_namespace}"
-		parent_link="base_link"
 		frame_id="world"
 		topic_name="/fix"
@@ -18,4 +18,5 @@
 		reference_heading="0"
 		reference_altitude="0"
+		parent="base_link"
 		has_inertia="true">
 	    <origin xyz="0 0 0" rpy="0 0 0" />
@@ -39,5 +40,4 @@
 		 frame_id
 		 topic_name
-		 parent_link
 		 velocity_topic_name
 		 reference_latitude
@@ -45,4 +45,5 @@
 		 reference_heading
 		 reference_altitude
+		 parent
 	     has_inertia
 	     *origin
@@ -51,21 +52,5 @@
 	     *inertial
 		">
-<link name="${name}_link">
-  <visual>
-      <xacro:insert_block name="geometry" />
-	  <xacro:insert_block name="material" />
-  </visual>
-  <collision name="${name}_collision">
-  	  	<xacro:insert_block name="geometry" />
-  </collision>
-  <xacro:if value="${has_inertia}">
-	<xacro:insert_block name="inertial" />
-  </xacro:if>
-</link>
-<joint name="${name}_joint" type="fixed">
-	<parent link="${parent_link}" />
-	<child link="${name}_link" />
-	<xacro:insert_block name="origin" />
-</joint>
+<xacro:rr_geo_ins/>
 <gazebo>
 	<plugin name="${name}_controller"

File: defs/test_robots/diff_drive_bot.xacro (robot description, xacro)
@@ -152,5 +152,4 @@
 		name="gps0"
 	 	robot_namespace="${robot_namespace}"
-		parent_link="base_link"
 		frame_id="world"
 		topic_name="/fix"
@@ -160,4 +159,5 @@
 		reference_heading="0"
 		reference_altitude="0"
+		parent="base_link"
 		has_inertia="true">
 	    <origin xyz="${-(chassis_len/2-0.04/2)} ${chassis_width/2-0.015}
@@ -174,7 +174,5 @@
 	    </xacro:inertia_box>
 	</xacro:rr_gps_receiver>
-	<gazebo reference="gps0">
-		<material value="Gazebo/FlatBlack" />
-	</gazebo>
+	<xacro:rr_gaz_mat_s name="gps0" material="Gazebo/FlatBlack"/>
 <!-- IMU -->
 <xacro:rr_imu
@@ -182,5 +180,4 @@
 	 	robot_namespace=""
 		topic_name="/imu"
-		parent_link="base_link"
 		gaussian_noise="2.89e-08"
 		imu_x="0"
@@ -190,4 +187,5 @@
 		imu_pitch="0"
 		imu_yaw="0"
+		parent="base_link"
 		has_inertia="false"
 		>
@@ -204,15 +202,9 @@
 		 <inertial/>
 	</xacro:rr_imu>
-<!-- CAMERA
+	<xacro:rr_gaz_mat_s name="imu0" material="Gazebo/Yellow"/>
+<!-- CAMERA  -->
 <xacro:rr_cam
 		name             ="cam0"
 	 	robot_namespace  ="${robot_namespace}"
-		parent_link      ="base_link"
-		x                ="${chassis_len/2}"
-	    y                ="0"
-        z                ="0"
-        roll             ="0"
-        pitch            ="-0.01"
-        yaw              ="0"
 		always_on        ="true"
 		frame_name       ="camera0"
@@ -233,5 +225,19 @@
 		dist_T2          ="0.0"
 		update_rate      ="30"
-        />	 -->
+		parent           ="base_link"
+	    has_inertia      ="false"
+		>
+		<origin xyz="${chassis_len/2}
+                     0
+		             ${chassis_center}" rpy="0 0 0" />
+		<geometry>
+			<box size="0.02 0.02 0.02" />
+		</geometry>
+		<material name="Yellow">
+			<color rgba="0 0 0 1"/>
+		</material>
+		 <inertial/>
+        </xacro:rr_cam>
+		<xacro:rr_gaz_mat_s name="cam0" material="Gazebo/FlatBlack"/>
 <!-- LIDAR
 <xacro:rplidar id="0"
