Commit message: change constant name of pi

File: defs/constants.xacro (robot description, xacro)
@@ -7,4 +7,4 @@
        <xacro:property name="debugLevel" value="1"/>
        <!-- Pi -->
-	   <xacro:property name="const_pi" value="3.1415926535897931"/>
+	   <xacro:property name="rr_const_pi" value="3.1415926535897931"/>
 </robot>

File: defs/drive/wheel_solid.xacro (robot description, xacro)
@@ -21,5 +21,5 @@
 		<inertial>
 			<mass value="${mass}"/>
-			<origin xyz="0 0 0" rpy="${const_pi/2} 0 0" />
+			<origin xyz="0 0 0" rpy="${rr_const_pi/2} 0 0" />
 		    <inertia  ixx="${1/4*mass*radius*radius+1/12*mass+width*width}"
                       iyy="${1/4*mass*radius*radius+1/12*mass+width*width}"
@@ -29,5 +29,5 @@
 		<visual>
 			<origin xyz="0 0 0"
-			        rpy="${const_pi/2} 0 0"/>
+			        rpy="${rr_const_pi/2} 0 0"/>
 			<geometry>
 				<cylinder radius="${radius}" length="${width}"/>
@@ -39,5 +39,5 @@
 		<collision>
 			<origin xyz="0 0 0"
-			        rpy="${const_pi/2} 0 0"/>
+			        rpy="${rr_const_pi/2} 0 0"/>
 			<geometry>
 				<cylinder radius="${radius}" length="${width}"/>
