Commit message: update laser remove robot namespace tags remove old sensor files change name of laser scanner file

File: defs/geometry/geo_ins.xacro (robot description, xacro)
@@ -19,5 +19,5 @@
 	  <xacro:insert_block name="material" />
 	</visual>
-	<collision name="${name}_collision">
+	<collision name="${name}_link_collision">
 	  	<xacro:insert_block name="geometry" />
 	</collision>

File: defs/rapid_robot.xacro (robot description, xacro)
@@ -18,6 +18,5 @@
 <!-- Sensors -->
 <xacro:include filename="$(find rapid_robot_xacros)/defs/sensors/contact/bumper.xacro"/>
-<xacro:include filename="$(find rapid_robot_xacros)/defs/sensors/distance/laser_scanner_2d.xacro"/>
-<xacro:include filename="$(find rapid_robot_xacros)/defs/sensors/distance/sonar.xacro"/>
+<xacro:include filename="$(find rapid_robot_xacros)/defs/sensors/distance/laser_2d.xacro"/>
 <xacro:include filename="$(find rapid_robot_xacros)/defs/sensors/imaging/camera.xacro"/>
 <xacro:include filename="$(find rapid_robot_xacros)/defs/sensors/inertia/imu.xacro"/>

File: defs/sensors/contact/bumper.xacro (robot description, xacro)
@@ -30,27 +30,11 @@
 <xacro:macro name="rr_bumper"
 	params="name parent always_on update_rate topic has_inertia *origin *geometry *material *inertial">
-	<link name="${name}">
-	  <visual>
-	      <xacro:insert_block name="geometry" />
-		  <xacro:insert_block name="material" />
-	  </visual>
-      <collision name="${name}_collision">
-	  	  	<xacro:insert_block name="geometry" />
-	  </collision>
-	  <xacro:if value="${has_inertia}">
-		<xacro:insert_block name="inertial" />
-	  </xacro:if>
-	</link>
-	<joint name="${name}_${parent}_joint" type="fixed">
-		<parent link="${parent}" />
-		<child link="${name}" />
-		<xacro:insert_block name="origin" />
-	</joint>
-	<gazebo reference="${name}">
+	<xacro:rr_geo_ins/>
+	<gazebo reference="${name}_link">
 	  <sensor name="${name}_sensor" type="contact">
 	    <always_on>${always_on}</always_on>
 	    <update_rate>${update_rate}</update_rate>
 	    <contact>
-	      <collision>${name}_collision</collision>
+	      <collision>${name}_link_collision</collision>
 	    </contact>
 	    <plugin name="${name}_plugin" filename="libgazebo_ros_bumper.so">

File: defs/sensors/distance/laser_2d.xacro (robot description, xacro)
@@ -5,23 +5,60 @@
        xmlns:xacro="http://ros.org/wiki/xacro"
 >
-<!-- Example -->
-<!--
-<xacro:rplidar id="0"
-	 	robot_namespace="${robot_namespace}"
-		topic_name="/laser/scan"
-		frame_name="laser"
-		parent_link="chassis"
-		x="0"
-        y="0"
-        z="${chassis_height/2}"
-	    roll="0"
-	    pitch="0"
-        yaw="0"
-		update_rate="5.5"
-		visualize="false" />
--->
-<xacro:include filename="$(find rapid_robot_xacros)/defs/constants.xacro"/>
+<xacro:macro name="rr_laser_2d" params="
+	name
+	topic_name
+	update_rate
+	visualize
+	hor_samples
+	hor_resolution
+	hor_min_angle
+	hor_max_angle
+	range_min
+	range_max
+	range_resolution
+	noise_type
+    noise_mean
+    noise_stddev
+	parent
+    has_inertia
+    *origin
+    *geometry
+    *material
+    *inertial
+	*laser_pose
+	">
+	<xacro:rr_geo_ins/>
+  <gazebo reference="${name}_link">
+    <sensor type="gpu_ray" name="${name}_sensor">
+      <visualize>${visualize}</visualize>
+      <update_rate>${update_rate}</update_rate>
+      <ray>
+        <scan>
+          <horizontal>
+            <samples>${hor_samples}</samples>
+            <resolution>${hor_resolution}</resolution>
+            <min_angle>${hor_min_angle}</min_angle>
+            <max_angle>${hor_max_angle}</max_angle>
+          </horizontal>
+        </scan>
+        <range>
+          <min>${range_min}</min>
+          <max>${range_max}</max>
+          <resolution>${range_resolution}</resolution>
+        </range>
+        <noise>
+          <type>${noise_type}</type>
+          <mean>${noise_mean}</mean>
+          <stddev>${noise_stddev}</stddev>
+        </noise>
+      </ray>
+      <plugin name="${name}_gpu_laser_controller" filename="libgazebo_ros_gpu_laser.so">
+      	<topicName>${topic_name}</topicName>
+        <frameName>${name}_link</frameName>
+      </plugin>
+    </sensor>
+  </gazebo>
+</xacro:macro>
 <xacro:macro name="rplidar" params="id
-								robot_namespace
 								topic_name
 								frame_name
@@ -31,5 +68,4 @@
 								visualize
 								">
- <xacro:property />
   <!-- RPLidar Laser -->
   <link name="rplidar${id}_link">
@@ -72,5 +108,5 @@
             <resolution>1</resolution>
             <min_angle>0</min_angle>
-            <max_angle>${2*const_pi}</max_angle>
+            <max_angle>${2*rr_const_pi}</max_angle>
           </horizontal>
         </scan>
@@ -87,5 +123,4 @@
       </ray>
       <plugin name="gazebo_ros_head_rplidar${id}_controller" filename="libgazebo_ros_gpu_laser.so">
-        <robotNamespace>${robot_namespace}</robotNamespace>
       	<topicName>${topic_name}</topicName>
         <frameName>rplidar${id}_link</frameName>

File: defs/sensors/inertia/imu.xacro (robot description, xacro)
@@ -36,5 +36,4 @@
 -->
 <xacro:macro name="rr_imu" params="name
-								robot_namespace
 								topic_name
 								gaussian_noise
@@ -55,5 +54,4 @@
 <gazebo>
 	  <plugin name="imu{id}_controller" filename="libgazebo_ros_imu.so">
-			<robotNamespace>${robot_namespace}</robotNamespace>
 			<bodyName>${name}_link</bodyName>
 			<topicName>${topic_name}</topicName>

File: defs/sensors/position/gps.xacro (robot description, xacro)
@@ -10,5 +10,4 @@
 	<xacro:rr_gps_receiver
 		name="gps0"
-	 	robot_namespace="${robot_namespace}"
 		frame_id="world"
 		topic_name="/fix"
@@ -37,5 +36,4 @@
 <xacro:macro name="rr_gps_receiver"
 params= "name
-		 robot_namespace
 		 frame_id
 		 topic_name
@@ -56,5 +54,4 @@
 	<plugin name="${name}_controller"
 		    filename="libhector_gazebo_ros_gps.so">
-		<robotNamespace>${robot_namespace}</robotNamespace>
 		<bodyName>${name}_link</bodyName>
 		<frameId>${frame_id}</frameId>

File: defs/test_robots/diff_drive_bot.xacro (robot description, xacro)
@@ -14,13 +14,12 @@
 <xacro:property name="wheel_base_center_x"     value="${chassis_len/(-1.618*3)}"       />
 <xacro:property name="caster_collision_x"      value="${chassis_len/(1.618*2)}"        />
-<xacro:property name="robot_namespace" value="/" />
-<xacro:property name="chassis_center" value="${chassis_floor_clearance+chassis_height/2}" />
+<xacro:property name="chassis_center_z" value="${chassis_floor_clearance+chassis_height/2}" />
 <!--CHASSIS-->
 <link name="base_link">
 	<xacro:rr_inertia_box_solid x="${chassis_len}" y="${chassis_width}" z="${chassis_height}" mass="1">
-      	 <origin xyz="0 0 ${chassis_center}" rpy="0 0 0" />
+      	 <origin xyz="-${-wheel_base_center_x} 0 ${chassis_center_z}" rpy="0 0 0" />
     </xacro:rr_inertia_box_solid>
 	<visual>
-		<origin xyz="0 0 ${chassis_center}" rpy="0 0 0" />
+		<origin xyz="${-wheel_base_center_x} 0 ${chassis_center_z}" rpy="0 0 0" />
 		<geometry>
 			<box size="${chassis_len} ${chassis_width} ${chassis_height}" />
@@ -29,5 +28,5 @@
 	</visual>
 	<collision>
-		<origin xyz="0 0 ${chassis_center}" rpy="0 0 0" />
+		<origin xyz="${-wheel_base_center_x} 0 ${chassis_center_z}" rpy="0 0 0" />
 		<geometry>
 			<box size="${chassis_len} ${chassis_width} ${chassis_height}" />
@@ -38,5 +37,5 @@
 <!-- Bumper -->
 <xacro:rr_bumper name="bumper0" parent="base_link" always_on="true" update_rate="30" topic="bumper0"  has_inertia="true">
-	<origin xyz="${chassis_len/2} ${chassis_width/2} ${chassis_center}" rpy="0 0 0" />
+	<origin xyz="${chassis_len/2-wheel_base_center_x} ${chassis_width/2} ${chassis_center_z}" rpy="0 0 0" />
 	<geometry>
 		<box size="0.02 0.02 ${chassis_height}" />
@@ -49,5 +48,5 @@
 <xacro:rr_m_gz_black name="bumper0"/>
 <xacro:rr_bumper name="bumper1" parent="base_link" always_on="true" update_rate="30" topic="bumper1"  has_inertia="true">
-	<origin xyz="${chassis_len/2} -${chassis_width/2} ${chassis_center}" rpy="0 0 0" />
+	<origin xyz="${chassis_len/2-wheel_base_center_x} -${chassis_width/2} ${chassis_center_z}" rpy="0 0 0" />
 	<geometry>
 		<box size="0.02 0.02 ${chassis_height}" />
@@ -60,5 +59,5 @@
 <xacro:rr_m_gz_black name="bumper1"/>
 <xacro:rr_bumper name="bumper2" parent="base_link" always_on="true" update_rate="30" topic="bumper2"  has_inertia="true">
-	<origin xyz="${chassis_len/2} 0 ${chassis_center-chassis_height/4}" rpy="0 0 0" />
+	<origin xyz="${chassis_len/2-wheel_base_center_x} 0 ${chassis_center_z-chassis_height/4}" rpy="0 0 0" />
 	<geometry>
 		<box size="0.02 ${chassis_width-0.04} 0.02" />
@@ -98,10 +97,10 @@
 	<parent link="base_link" />
 	<child link="caster_collision" />
-	<origin xyz="${caster_collision_x} 0 ${chassis_center-(chassis_height/2)}" rpy="0 0 0" />
+	<origin xyz="${caster_collision_x-wheel_base_center_x} 0 ${chassis_center_z-(chassis_height/2)}" rpy="0 0 0" />
 </joint>
 <!-- Drive -->
 <xacro:rr_diff_drive
 	 base_frame="base_link"
-	 wheel_base_center_x="${wheel_base_center_x}"
+	 wheel_base_center_x="0"
      wheel_separation ="${chassis_width}"
      wheel_diameter="${wheel_diameter}"
@@ -116,5 +115,5 @@
      wheel_contact_stiffness="1000000.0"
 	 wheel_mass="3"
-	 z_dist="${chassis_center-((chassis_floor_clearance+chassis_height/2)-(wheel_diameter/2))}"
+	 z_dist="${chassis_center_z-((chassis_floor_clearance+chassis_height/2)-(wheel_diameter/2))}"
      cmd_topic="/cmd_vel"
 	 odom_topic="odom"
@@ -130,5 +129,4 @@
 	<xacro:rr_gps_receiver
 		name="gps0"
-	 	robot_namespace="${robot_namespace}"
 		frame_id="world"
 		topic_name="/fix"
@@ -140,6 +138,6 @@
 		parent="base_link"
 		has_inertia="true">
-	    <origin xyz="${-(chassis_len/2-0.04/2)} ${chassis_width/2-0.015}
-                     ${chassis_center+chassis_height/2+0.02/2}"
+	    <origin xyz="${-(chassis_len/2-0.04/2)-wheel_base_center_x} ${chassis_width/2-0.015}
+                     ${chassis_center_z+chassis_height/2+0.02/2}"
 	                 rpy="0 0 0" />
 		<geometry>
@@ -157,5 +155,4 @@
 <xacro:rr_imu
 		name="imu0"
-	 	robot_namespace=""
 		topic_name="/imu"
 		gaussian_noise="2.89e-08"
@@ -169,7 +166,6 @@
 		has_inertia="false"
 		>
-		<origin xyz="${wheel_base_center_x}
-                       0
-		             ${chassis_center-((chassis_floor_clearance+
+		<origin xyz="0 0
+		             ${chassis_center_z-((chassis_floor_clearance+
                        chassis_height/2)-(wheel_diameter/2))}" rpy="0 0 0" />
 		<geometry>
@@ -206,7 +202,7 @@
 	    has_inertia      ="false"
 		>
-		<origin xyz="${chassis_len/2}
+		<origin xyz="${chassis_len/2-wheel_base_center_x}
                      0
-		             ${chassis_center}" rpy="0 0 0" />
+		             ${chassis_center_z}" rpy="0 0 0" />
 		<geometry>
 			<box size="0.02 0.02 0.02" />
@@ -218,18 +214,33 @@
         </xacro:rr_cam>
 		<xacro:rr_gaz_mat_s name="cam0" material="Gazebo/FlatBlack"/>
-<!-- LIDAR
-<xacro:rplidar id="0"
-	 	robot_namespace="${robot_namespace}"
-		topic_name="/laser/scan"
-		frame_name="laser"
-		parent_link="base_link"
-		x="0"
-        y="0"
-        z="${chassis_height/2}"
-	    roll="0"
-	    pitch="0"
-        yaw="0"
-		update_rate="5.5"
-		visualize="false" />
- -->
+<!-- LIDAR -->
+<xacro:rr_laser_2d
+	name="laser"
+	topic_name="scan/laser"
+	update_rate="5.5"
+	visualize="false"
+	hor_samples="360"
+	hor_resolution="1"
+	hor_min_angle="${0}"
+	hor_max_angle="${2*rr_const_pi}"
+	range_min="0.20"
+	range_max="6"
+	range_resolution="0.005"
+	noise_type="gaussian"
+    noise_mean="0.0"
+    noise_stddev="0.01"
+	parent="base_link"
+    has_inertia="false"
+	>
+	<origin xyz="0 0 ${chassis_center_z+chassis_height/2+0.1/2}" rpy="0 0 0" />
+	<geometry>
+		<box size="0.098 0.07 0.1" />
+	</geometry>
+	<material name="Black">
+		<color rgba="0 0 0 1"/>
+	</material>
+	<inertial/>
+    <pose>0 0 0 0 0 0</pose>
+</xacro:rr_laser_2d>
+<xacro:rr_gaz_mat_s name="laser" material="Gazebo/FlatBlack"/>
 </robot>
