Commit message: add color macros (unfinished)

File: defs/material/gazebo_simple.xacro (robot description, xacro)
@@ -4,8 +4,21 @@
        xmlns:interface="http://playerstage.sourceforge.net/gazebo/xmlschema/#interface"
        xmlns:xacro="http://ros.org/wiki/xacro">
-<xacro:macro name="rr_gaz_mat_s" params="name material">
-   <gazebo reference="${name}_link">
+<xacro:macro name="rr_mat_gaz" params="name material">
+   <gazebo reference="${link}_link">
 	<material value="${material}" />
    </gazebo>
 </xacro:macro>
+<xacro:macro name="rr_mat_color_def" params="color rgba">
+	<material name="rr_m_${color}">
+		<color rgba="${rgba}"/>
+	</material>
+</xacro:macro>
+<!-- predefine color macro -->
+<xacro:macro name="rr_mat_gaz_color_def" params="color material">
+<!--	<xacro:macro name="rr_mat_gaz_${color}" params="name material">
+	   <gazebo reference="${name}_link">
+		<material value="${material}" />
+	   </gazebo>
+	</xacro:macro>-->
+</xacro:macro>
 </robot>

File: defs/rapid_robot.xacro (robot description, xacro)
@@ -10,4 +10,5 @@
 <!-- Material -->
 <xacro:include filename="$(find rapid_robot_xacros)/defs/material/gazebo_simple.xacro"/>
+<xacro:include filename="$(find rapid_robot_xacros)/defs/material/rr_mats.xacro"/>
 <!-- Inertia -->
 <xacro:include filename="$(find rapid_robot_xacros)/defs/inertia/box_solid.xacro"/>

File: defs/test_robots/diff_drive_bot.xacro (robot description, xacro)
@@ -26,7 +26,5 @@
 			<box size="${chassis_len} ${chassis_width} ${chassis_height}" />
 		</geometry>
-		<material name="Green">
-			<color rgba="0 1 0 0.5"/>
-		</material>
+		<material name="rr_m_green_tp"/>
 	</visual>
 	<collision>
@@ -37,7 +35,5 @@
 	</collision>
 </link>
-<gazebo reference="base_link">
-	<material value="Gazebo/Green"/>
-</gazebo>
+<xacro:rr_m_gz_green name="base_link"/>
 <!-- Bumper -->
 <xacro:rr_bumper name="bumper0" parent="base_link" always_on="true" update_rate="30" topic="bumper0"  has_inertia="true">
@@ -46,14 +42,10 @@
 		<box size="0.02 0.02 ${chassis_height}" />
 	</geometry>
-	<material name="Black">
-		<color rgba="0 0 0 1"/>
-	</material>
+	<material name="rr_m_black"/>
 	 <xacro:rr_inertia_box_solid x="0.02" y="0.02" z="${chassis_height}" mass="0.1">
       <origin xyz="0 0 0" rpy="0 0 0" />
     </xacro:rr_inertia_box_solid>
 </xacro:rr_bumper>
-<gazebo reference="bumper0">
-	<material value="Gazebo/FlatBlack" />
-</gazebo>
+<xacro:rr_m_gz_black name="bumper0"/>
 <xacro:rr_bumper name="bumper1" parent="base_link" always_on="true" update_rate="30" topic="bumper1"  has_inertia="true">
 	<origin xyz="${chassis_len/2} -${chassis_width/2} ${chassis_center}" rpy="0 0 0" />
@@ -61,14 +53,10 @@
 		<box size="0.02 0.02 ${chassis_height}" />
 	</geometry>
-	<material name="Black">
-		<color rgba="0 0 0 1"/>
-	</material>
+	<material name="rr_m_black"/>
 	 <xacro:inertia_box x="0.02" y="0.02" z="${chassis_height}" mass="0.1">
       <origin xyz="0 0 0" rpy="0 0 0" />
     </xacro:inertia_box>
 </xacro:rr_bumper>
-<gazebo reference="bumper1">
-	<material value="Gazebo/FlatBlack" />
-</gazebo>
+<xacro:rr_m_gz_black name="bumper1"/>
 <xacro:rr_bumper name="bumper2" parent="base_link" always_on="true" update_rate="30" topic="bumper2"  has_inertia="true">
 	<origin xyz="${chassis_len/2} 0 ${chassis_center-chassis_height/4}" rpy="0 0 0" />
@@ -76,14 +64,10 @@
 		<box size="0.02 ${chassis_width-0.04} 0.02" />
 	</geometry>
-	<material name="Black">
-		<color rgba="0 0 0 1"/>
-	</material>
+	<material name="rr_m_black"/>
 	 <xacro:inertia_box x="0.02" y="0.02" z="0.04" mass="0.1">
       <origin xyz="0 0 0" rpy="0 0 0" />
     </xacro:inertia_box>
 </xacro:rr_bumper>
-<gazebo reference="bumper2">
-	<material value="Gazebo/FlatBlack" />
-</gazebo>
+<xacro:rr_m_gz_black name="bumper2"/>
 <!--CASTER -->
 <link name="caster_collision">
@@ -92,7 +76,5 @@
 			<sphere radius="${chassis_floor_clearance}" />
 		</geometry>
-		<material name="Black">
-			<color rgba="0 0 0 1"/>
-		</material>
+		<material name="rr_m_black"/>
 	</visual>
 	<collision>
@@ -112,7 +94,5 @@
     </inertial>
 </link>
-<gazebo reference="caster_collision">
-	<material value="Gazebo/FlatBlack"/>
-</gazebo>
+<xacro:rr_m_gz_black name="caster_collision"/>
 <joint name="base_caster_col_joint" type="fixed">
 	<parent link="base_link" />

Commit message: create colors manually, fix colors of sensors and chassis

File: defs/material/gazebo_simple.xacro (robot description, xacro)
@@ -14,11 +14,3 @@
 	</material>
 </xacro:macro>
-<!-- predefine color macro -->
-<xacro:macro name="rr_mat_gaz_color_def" params="color material">
-<!--	<xacro:macro name="rr_mat_gaz_${color}" params="name material">
-	   <gazebo reference="${name}_link">
-		<material value="${material}" />
-	   </gazebo>
-	</xacro:macro>-->
-</xacro:macro>
 </robot>

File: defs/material/rr_mats.xacro (robot description, xacro)
@@ -5,6 +5,14 @@
        xmlns:xacro="http://ros.org/wiki/xacro">
 <!-- Gazebo Colors -->
-<xacro:rr_mat_gaz_color_def color="green" material="Gazebo/Green" />
-<xacro:rr_mat_gaz_color_def color="black" material="Gazebo/FlatBlack" />
+<xacro:macro name="rr_m_gz_green" params="name">
+	<gazebo reference="${name}_link">
+	<material value="Gazebo/Green" />
+   </gazebo>
+</xacro:macro>
+<xacro:macro name="rr_m_gz_black" params="name">
+	<gazebo reference="${name}_link">
+	<material value="Gazebo/FlatBlack" />
+   </gazebo>
+</xacro:macro>
 <!-- URDF colors -->
 <xacro:rr_mat_color_def color="green" rgba="0 1 0 1" />

File: defs/test_robots/diff_drive_bot/chassis.xacro (robot description, xacro)
@@ -23,4 +23,4 @@
 	</collision>
 </link>
-<xacro:rr_m_gz_green name="base_link"/>
+<xacro:rr_m_gz_green name="base"/>
 </robot>

File: defs/test_robots/diff_drive_bot/laser.xacro (robot description, xacro)
@@ -32,4 +32,4 @@
     <pose>0 0 0 0 0 0</pose>
 </xacro:rr_laser_2d>
-<xacro:rr_gaz_mat_s name="laser" material="Gazebo/FlatBlack"/>
+<xacro:rr_m_gz_black name="laser"/>
 </robot>
