Commit message: fix color of camera

File: defs/test_robots/diff_drive_bot.xacro (robot description, xacro)
@@ -234,5 +234,5 @@
 			<box size="0.02 0.02 0.02" />
 		</geometry>
-		<material name="Yellow">
+		<material name="Black">
 			<color rgba="0 0 0 1"/>
 		</material>

Commit message: split test bot into include files

File: defs/test_robots/diff_drive_bot.xacro (robot description, xacro)
@@ -15,232 +15,10 @@
 <xacro:property name="caster_collision_x"      value="${chassis_len/(1.618*2)}"        />
 <xacro:property name="chassis_center_z" value="${chassis_floor_clearance+chassis_height/2}" />
-<!--CHASSIS-->
-<link name="base_link">
-	<xacro:rr_inertia_box_solid x="${chassis_len}" y="${chassis_width}" z="${chassis_height}" mass="1">
-      	 <origin xyz="-${-wheel_base_center_x} 0 ${chassis_center_z}" rpy="0 0 0" />
-    </xacro:rr_inertia_box_solid>
-	<visual>
-		<origin xyz="${-wheel_base_center_x} 0 ${chassis_center_z}" rpy="0 0 0" />
-		<geometry>
-			<box size="${chassis_len} ${chassis_width} ${chassis_height}" />
-		</geometry>
-		<material name="rr_m_green_tp"/>
-	</visual>
-	<collision>
-		<origin xyz="${-wheel_base_center_x} 0 ${chassis_center_z}" rpy="0 0 0" />
-		<geometry>
-			<box size="${chassis_len} ${chassis_width} ${chassis_height}" />
-		</geometry>
-	</collision>
-</link>
-<xacro:rr_m_gz_green name="base_link"/>
-<!-- Bumper -->
-<xacro:rr_bumper name="bumper0" parent="base_link" always_on="true" update_rate="30" topic="bumper0"  has_inertia="true">
-	<origin xyz="${chassis_len/2-wheel_base_center_x} ${chassis_width/2} ${chassis_center_z}" rpy="0 0 0" />
-	<geometry>
-		<box size="0.02 0.02 ${chassis_height}" />
-	</geometry>
-	<material name="rr_m_black"/>
-	 <xacro:rr_inertia_box_solid x="0.02" y="0.02" z="${chassis_height}" mass="0.1">
-      <origin xyz="0 0 0" rpy="0 0 0" />
-    </xacro:rr_inertia_box_solid>
-</xacro:rr_bumper>
-<xacro:rr_m_gz_black name="bumper0"/>
-<xacro:rr_bumper name="bumper1" parent="base_link" always_on="true" update_rate="30" topic="bumper1"  has_inertia="true">
-	<origin xyz="${chassis_len/2-wheel_base_center_x} -${chassis_width/2} ${chassis_center_z}" rpy="0 0 0" />
-	<geometry>
-		<box size="0.02 0.02 ${chassis_height}" />
-	</geometry>
-	<material name="rr_m_black"/>
-	 <xacro:inertia_box x="0.02" y="0.02" z="${chassis_height}" mass="0.1">
-      <origin xyz="0 0 0" rpy="0 0 0" />
-    </xacro:inertia_box>
-</xacro:rr_bumper>
-<xacro:rr_m_gz_black name="bumper1"/>
-<xacro:rr_bumper name="bumper2" parent="base_link" always_on="true" update_rate="30" topic="bumper2"  has_inertia="true">
-	<origin xyz="${chassis_len/2-wheel_base_center_x} 0 ${chassis_center_z-chassis_height/4}" rpy="0 0 0" />
-	<geometry>
-		<box size="0.02 ${chassis_width-0.04} 0.02" />
-	</geometry>
-	<material name="rr_m_black"/>
-	 <xacro:inertia_box x="0.02" y="0.02" z="0.04" mass="0.1">
-      <origin xyz="0 0 0" rpy="0 0 0" />
-    </xacro:inertia_box>
-</xacro:rr_bumper>
-<xacro:rr_m_gz_black name="bumper2"/>
-<!--CASTER -->
-<link name="caster_collision">
-	<visual>
-		<geometry>
-			<sphere radius="${chassis_floor_clearance}" />
-		</geometry>
-		<material name="rr_m_black"/>
-	</visual>
-	<collision>
-		<geometry>
-			<sphere radius="${chassis_floor_clearance}" />
-		</geometry>
-	</collision>
-    <inertial>
-    <mass value="1.0"/>
-    <origin xyz="0.0 0.0 0.0"/>
-    <inertia ixx="0.1"
-             iyy="0.1"
-             izz="0.1"
-        	 iyz="0.0"
-             ixy="0.0"
-             ixz="0.0"/>
-    </inertial>
-</link>
-<xacro:rr_m_gz_black name="caster_collision"/>
-<joint name="base_caster_col_joint" type="fixed">
-	<parent link="base_link" />
-	<child link="caster_collision" />
-	<origin xyz="${caster_collision_x-wheel_base_center_x} 0 ${chassis_center_z-(chassis_height/2)}" rpy="0 0 0" />
-</joint>
-<!-- Drive -->
-<xacro:rr_diff_drive
-	 base_frame="base_link"
-	 wheel_base_center_x="0"
-     wheel_separation ="${chassis_width}"
-     wheel_diameter="${wheel_diameter}"
-	 wheel_width="${wheel_width}"
-     wheel_torque="5"
-	 wheel_acceleration="1"
-	 wheel_joint_limit_vel="2"
-	 wheel_joint_limit_effort="2"
-	 wheel_friction1="100000"
-     wheel_friction2="1000"
-	 wheel_contact_damping="100.0"
-     wheel_contact_stiffness="1000000.0"
-	 wheel_mass="3"
-	 z_dist="${chassis_center_z-((chassis_floor_clearance+chassis_height/2)-(wheel_diameter/2))}"
-     cmd_topic="/cmd_vel"
-	 odom_topic="odom"
-     odom_frame="odom"
-	 ros_plugin_always_on="true"
-	 ros_plugin_controller_name="diff_drv0"
-     ros_plugin_update_rate="100"
-	 ros_plugin_odom_source="encoder"
-	 ros_plugin_publish_wheel_joint_state="true"
-	 ros_plugin_publish_wheel_tf="true"
-	 ros_plugin_publish_tf="1" />
-<!-- GPS -->
-	<xacro:rr_gps_receiver
-		name="gps0"
-		frame_id="world"
-		topic_name="/fix"
-		velocity_topic_name="/fix_vel"
-		reference_latitude="49"
-		reference_longitude="8"
-		reference_heading="0"
-		reference_altitude="0"
-		parent="base_link"
-		has_inertia="true">
-	    <origin xyz="${-(chassis_len/2-0.04/2)-wheel_base_center_x} ${chassis_width/2-0.015}
-                     ${chassis_center_z+chassis_height/2+0.02/2}"
-	                 rpy="0 0 0" />
-		<geometry>
-			<box size="0.04 0.03 0.02" />
-		</geometry>
-		<material name="Black">
-			<color rgba="0 0 0 1"/>
-		</material>
-		 <xacro:inertia_box x="0.02" y="0.02" z="0.04" mass="0.1">
-	      <origin xyz="0 0 0" rpy="0 0 0" />
-	    </xacro:inertia_box>
-	</xacro:rr_gps_receiver>
-	<xacro:rr_gaz_mat_s name="gps0" material="Gazebo/FlatBlack"/>
-<!-- IMU -->
-<xacro:rr_imu
-		name="imu0"
-		topic_name="/imu"
-		gaussian_noise="2.89e-08"
-		imu_x="0"
-		imu_y="0"
-		imu_z="0"
-		imu_roll="0"
-		imu_pitch="0"
-		imu_yaw="0"
-		parent="base_link"
-		has_inertia="false"
-		>
-		<origin xyz="0 0
-		             ${chassis_center_z-((chassis_floor_clearance+
-                       chassis_height/2)-(wheel_diameter/2))}" rpy="0 0 0" />
-		<geometry>
-			<box size="0.02 0.02 0.02" />
-		</geometry>
-		<material name="Yellow">
-			<color rgba="1 1 0 1"/>
-		</material>
-		 <inertial/>
-	</xacro:rr_imu>
-	<xacro:rr_gaz_mat_s name="imu0" material="Gazebo/Yellow"/>
-<!-- CAMERA  -->
-<xacro:rr_cam
-		name             ="cam0"
-		always_on        ="true"
-		frame_name       ="camera0"
-		image_width      ="640"
-		image_height     ="480"
-		image_format     ="R8G8B8"
-		clip_near        ="0.02"
-		clip_far         ="300"
-		noise_type       ="gaussian"
-		noise_mean       ="0.0"
-		noise_std_dev    ="0.007"
-		fov              ="0.873"
-		hack_baseline    ="0.07"
-		dist_K1          ="0.0"
-		dist_K2          ="0.0"
-		dist_K3          ="0.0"
-		dist_T1          ="0.0"
-		dist_T2          ="0.0"
-		update_rate      ="30"
-		parent           ="base_link"
-	    has_inertia      ="false"
-		>
-		<origin xyz="${chassis_len/2-wheel_base_center_x}
-                     0
-		             ${chassis_center_z}" rpy="0 0 0" />
-		<geometry>
-			<box size="0.02 0.02 0.02" />
-		</geometry>
-		<material name="Black">
-			<color rgba="0 0 0 1"/>
-		</material>
-		 <inertial/>
-        </xacro:rr_cam>
-		<xacro:rr_gaz_mat_s name="cam0" material="Gazebo/FlatBlack"/>
-<!-- LIDAR -->
-<xacro:rr_laser_2d
-	name="laser"
-	topic_name="scan/laser"
-	update_rate="5.5"
-	visualize="false"
-	hor_samples="360"
-	hor_resolution="1"
-	hor_min_angle="${0}"
-	hor_max_angle="${2*rr_const_pi}"
-	range_min="0.20"
-	range_max="6"
-	range_resolution="0.005"
-	noise_type="gaussian"
-    noise_mean="0.0"
-    noise_stddev="0.01"
-	parent="base_link"
-    has_inertia="false"
-	>
-	<origin xyz="0 0 ${chassis_center_z+chassis_height/2+0.1/2}" rpy="0 0 0" />
-	<geometry>
-		<box size="0.098 0.07 0.1" />
-	</geometry>
-	<material name="Black">
-		<color rgba="0 0 0 1"/>
-	</material>
-	<inertial/>
-    <pose>0 0 0 0 0 0</pose>
-</xacro:rr_laser_2d>
-<xacro:rr_gaz_mat_s name="laser" material="Gazebo/FlatBlack"/>
+<xacro:include filename="$(find rapid_robot_xacros)/defs/test_robots/diff_drive_bot/chassis.xacro"/>
+<xacro:include filename="$(find rapid_robot_xacros)/defs/test_robots/diff_drive_bot/bumpers.xacro"/>
+<xacro:include filename="$(find rapid_robot_xacros)/defs/test_robots/diff_drive_bot/caster.xacro"/>
+<xacro:include filename="$(find rapid_robot_xacros)/defs/test_robots/diff_drive_bot/drive.xacro"/>
+<xacro:include filename="$(find rapid_robot_xacros)/defs/test_robots/diff_drive_bot/imu.xacro"/>
+<xacro:include filename="$(find rapid_robot_xacros)/defs/test_robots/diff_drive_bot/camera.xacro"/>
+<xacro:include filename="$(find rapid_robot_xacros)/defs/test_robots/diff_drive_bot/laser.xacro"/>
 </robot>

Commit message: move properties to external file

File: defs/test_robots/diff_drive_bot.xacro (robot description, xacro)
@@ -5,14 +5,5 @@
        xmlns:xacro="http://ros.org/wiki/xacro" name="diff_drive_bot">
 <xacro:include filename="$(find rapid_robot_xacros)/defs/rapid_robot.xacro"/>
-<!-- Simple Robot Settings -->
-<xacro:property name="chassis_height"          value="0.25"                            />
-<xacro:property name="chassis_width"           value="${chassis_height*1.618}"         />
-<xacro:property name="chassis_len"             value="${chassis_width+chassis_height}" />
-<xacro:property name="chassis_floor_clearance" value="${chassis_height/(1.618*2)}"     />
-<xacro:property name="wheel_diameter"          value="${chassis_len/(1.618*1.618)}"    />
-<xacro:property name="wheel_width"             value="${chassis_width/(16.18)}"        />
-<xacro:property name="wheel_base_center_x"     value="${chassis_len/(-1.618*3)}"       />
-<xacro:property name="caster_collision_x"      value="${chassis_len/(1.618*2)}"        />
-<xacro:property name="chassis_center_z" value="${chassis_floor_clearance+chassis_height/2}" />
+<xacro:include filename="$(find rapid_robot_xacros)/defs/test_robots/diff_drive_bot/properties.xacro"/>
 <xacro:include filename="$(find rapid_robot_xacros)/defs/test_robots/diff_drive_bot/chassis.xacro"/>
 <xacro:include filename="$(find rapid_robot_xacros)/defs/test_robots/diff_drive_bot/bumpers.xacro"/>
