Commit message: rename caster dummy

File: defs/test_robots/diff_drive_bot/caster.xacro (robot description, xacro)
@@ -4,5 +4,5 @@
        xmlns:interface="http://playerstage.sourceforge.net/gazebo/xmlschema/#interface"
        xmlns:xacro="http://ros.org/wiki/xacro">
-<link name="caster_collision">
+<link name="caster_link">
 	<visual>
 		<geometry>
@@ -27,9 +27,9 @@
     </inertial>
 </link>
-<xacro:rr_m_gz_black name="caster_collision"/>
+<xacro:rr_m_gz_black name="caster"/>
 <joint name="base_caster_col_joint" type="fixed">
 	<parent link="base_link" />
-	<child link="caster_collision" />
-	<origin xyz="${caster_collision_x-wheel_base_center_x} 0 ${chassis_center_z-(chassis_height/2)}" rpy="0 0 0" />
+	<child link="caster_link" />
+	<origin xyz="${caster_x-wheel_base_center_x} 0 ${chassis_center_z-(chassis_height/2)}" rpy="0 0 0" />
 </joint>
 </robot>

File: defs/test_robots/diff_drive_bot/properties.xacro (robot description, xacro)
@@ -12,5 +12,5 @@
 <xacro:property name="wheel_width" value="${chassis_width/(16.18)}" />
 <xacro:property name="wheel_base_center_x" value="${chassis_len/(-1.618*3)}" />
-<xacro:property name="caster_collision_x" value="${chassis_len/(1.618*2)}"/>
+<xacro:property name="caster_x" value="${chassis_len/(1.618*2)}"/>
 <xacro:property name="chassis_center_z"
 				value="${chassis_floor_clearance+chassis_height/2}" />

Commit message: use inertia macro for caster sphere

File: defs/test_robots/diff_drive_bot/caster.xacro (robot description, xacro)
@@ -16,14 +16,7 @@
 		</geometry>
 	</collision>
-    <inertial>
-    <mass value="1.0"/>
-    <origin xyz="0.0 0.0 0.0"/>
-    <inertia ixx="0.1"
-             iyy="0.1"
-             izz="0.1"
-        	 iyz="0.0"
-             ixy="0.0"
-             ixz="0.0"/>
-    </inertial>
+    <xacro:rr_inertia_sphere_solid radius="${chassis_floor_clearance}" mass="0.2">
+    	<origin xyz="0 0 0" rpy="0 0 0"/>
+    </xacro:rr_inertia_sphere_solid>
 </link>
 <xacro:rr_m_gz_black name="caster"/>
