Commit message: fix problem, make robot spawn

File: defs/drive/diff_drive.xacro (robot description, xacro)
@@ -5,6 +5,6 @@
        xmlns:xacro="http://ros.org/wiki/xacro">
 <xacro:include filename="$(find rapid_robot_xacros)/defs/constants.xacro"/>
-<xacro:include filename="$(find rapid_robot_xacros)/defs/drive/simple_wheel.xacro"/>
-<xacro:macro name="diff_drive_setup"
+<xacro:include filename="$(find rapid_robot_xacros)/defs/drive/wheel_solid.xacro"/>
+<xacro:macro name="rr_diff_drive"
 	         params="base_frame
 					 robot_namespace
@@ -34,5 +34,5 @@
 					 ros_plugin_publish_tf
 	                 ">
-		<xacro:diff_drive_wheel
+		<xacro:rr_wheel_solid
 			                 name="${ros_plugin_controller_name}_wheel_left"
 						     base_frame="${base_frame}"
@@ -50,5 +50,5 @@
 							 friction2="${wheel_friction2}"
 							 />
-		<xacro:diff_drive_wheel
+		<xacro:rr_wheel_solid
                  name="${ros_plugin_controller_name}_wheel_right"
 			     base_frame="${base_frame}"

File: defs/drive/wheel_solid.xacro (robot description, xacro)
@@ -5,5 +5,5 @@
        xmlns:xacro="http://ros.org/wiki/xacro">
 	<xacro:include filename="$(find rapid_robot_xacros)/defs/constants.xacro"/>
-	<xacro:macro name="simple_full_wheel"
+	<xacro:macro name="rr_wheel_solid"
 			         params="name
 						     base_frame

File: defs/rapid_robot.xacro (robot description, xacro)
@@ -3,5 +3,5 @@
        xmlns:controller="http://playerstage.sourceforge.net/gazebo/xmlschema/#controller"
        xmlns:interface="http://playerstage.sourceforge.net/gazebo/xmlschema/#interface"
-       xmlns:xacro="http://ros.org/wiki/xacro" name="reppy_bot">
+       xmlns:xacro="http://ros.org/wiki/xacro">
 <!-- Constants -->
 <xacro:include filename="$(find rapid_robot_xacros)/defs/constants.xacro"/>
@@ -20,5 +20,5 @@
 <xacro:include filename="$(find rapid_robot_xacros)/defs/sensors/position/gps.xacro"/>
 <!-- Drives -->
-<xacro:include filename="$(find rapid_robot_xacros)/defs/drive/simple_wheel.xacro" />
+<xacro:include filename="$(find rapid_robot_xacros)/defs/drive/wheel_solid.xacro" />
 <xacro:include filename="$(find rapid_robot_xacros)/defs/drive/diff_drive.xacro" />
 </robot>

File: defs/test_robots/diff_drive_bot.xacro (robot description, xacro)
@@ -53,5 +53,5 @@
 	<material value="Gazebo/FlatBlack" />
 </gazebo>
-<xacro:rr_bumper name="bumper1" parent="chassis" always_on="true" update_rate="30" topic="bumper0"  has_inertia="true">
+<xacro:rr_bumper name="bumper1" parent="chassis" always_on="true" update_rate="30" topic="bumper1"  has_inertia="true">
 	<origin xyz="${chassis_len/2} -${chassis_width/2} 0" rpy="0 0 0" />
 	<geometry>
@@ -68,5 +68,5 @@
 	<material value="Gazebo/FlatBlack" />
 </gazebo>
-<xacro:rr_bumper name="bumper2" parent="chassis" always_on="true" update_rate="30" topic="bumper0"  has_inertia="true">
+<xacro:rr_bumper name="bumper2" parent="chassis" always_on="true" update_rate="30" topic="bumper2"  has_inertia="true">
 	<origin xyz="${chassis_len/2} 0 -${chassis_height/4}" rpy="0 0 0" />
 	<geometry>
@@ -117,3 +117,31 @@
 	<origin xyz="${caster_collision_x} 0 ${-(chassis_height/2)}" rpy="0 0 0" />
 </joint>
+<!-- Drive -->
+<xacro:rr_diff_drive
+	 base_frame="chassis"
+	 robot_namespace="${robot_namespace}"
+	 wheel_base_center_x="${wheel_base_center_x}"
+     wheel_separation ="${chassis_width}"
+     wheel_diameter="${wheel_diameter}"
+	 wheel_width="${wheel_width}"
+     wheel_torque="5"
+	 wheel_acceleration="1"
+	 wheel_joint_limit_vel="2"
+	 wheel_joint_limit_effort="2"
+	 wheel_friction1="100000"
+     wheel_friction2="1000"
+	 wheel_contact_damping="100.0"
+     wheel_contact_stiffness="1000000.0"
+	 wheel_mass="3"
+	 z_dist="${-((chassis_floor_clearance+chassis_height/2)-(wheel_diameter/2))}"
+     cmd_topic="/cmd_vel"
+	 odom_topic="odom"
+     odom_frame="odom"
+	 ros_plugin_always_on="true"
+	 ros_plugin_controller_name="diff_drv0"
+     ros_plugin_update_rate="100"
+	 ros_plugin_odom_source="encoder"
+	 ros_plugin_publish_wheel_joint_state="true"
+	 ros_plugin_publish_wheel_tf="true"
+	 ros_plugin_publish_tf="1" />
 </robot>

Commit message: change formatting rename base_frame to parent

File: defs/drive/diff_drive.xacro (robot description, xacro)
@@ -7,83 +7,84 @@
 <xacro:include filename="$(find rapid_robot_xacros)/defs/drive/wheel_solid.xacro"/>
 <xacro:macro name="rr_diff_drive"
-	         params="base_frame
-	                 wheel_base_center_x
-	                 wheel_separation
-	                 wheel_diameter
-	                 wheel_torque
-					 wheel_acceleration
-					 wheel_joint_limit_vel
-					 wheel_joint_limit_effort
-					 wheel_friction1
-	                 wheel_friction2
-	  				 wheel_contact_damping
-	                 wheel_contact_stiffness
-	 				 wheel_mass
-					 wheel_width
-					 z_dist
-	                 cmd_topic
-					 odom_topic
-	                 odom_frame
-					 ros_plugin_always_on
-					 ros_plugin_controller_name
-	                 ros_plugin_update_rate
-					 ros_plugin_odom_source
-					 ros_plugin_publish_wheel_joint_state
-					 ros_plugin_publish_wheel_tf
-					 ros_plugin_publish_tf
-	                 ">
-		<xacro:rr_wheel_solid
-			                 name="${ros_plugin_controller_name}_wheel_left"
-						     base_frame="${base_frame}"
-			                 radius="${wheel_diameter/2}"
-			                 width="${wheel_width}"
-							 mass="${wheel_mass}"
-							 origin_x="${wheel_base_center_x}"
-							 origin_y="${-(wheel_separation+wheel_width)/2}"
-							 origin_z="${z_dist}"
-							 limit_vel="${wheel_joint_limit_vel}"
-							 limit_effort="${wheel_joint_limit_effort}"
-							 contact_stiffness="${wheel_contact_stiffness}"
-							 contact_damping="${wheel_contact_damping}"
-		                     friction1="${wheel_friction1}"
-							 friction2="${wheel_friction2}"
-							 />
-		<xacro:rr_wheel_solid
-                 name="${ros_plugin_controller_name}_wheel_right"
-			     base_frame="${base_frame}"
-                 radius="${wheel_diameter/2}"
-                 width="${wheel_width}"
-				 mass="${wheel_mass}"
-				 origin_x="${wheel_base_center_x}"
-				 origin_y="${(wheel_separation+wheel_width)/2}"
-				 origin_z="${z_dist}"
-				 limit_vel="${wheel_joint_limit_vel}"
-				 limit_effort="${wheel_joint_limit_effort}"
-				 contact_stiffness="${wheel_contact_stiffness}"
-				 contact_damping="${wheel_contact_damping}"
-                 friction1="${wheel_friction1}"
-				 friction2="${wheel_friction2}"
-				 />
-	<gazebo>
-		<plugin name="${ros_plugin_controller_name}" filename="libgazebo_ros_diff_drive.so">
-			<robotBaseFrame>${base_frame}</robotBaseFrame>
-			<wheelSeparation>${wheel_separation}</wheelSeparation>
-			<wheelDiameter>${wheel_diameter}</wheelDiameter>
-			<wheelTorque>${wheel_torque}</wheelTorque>
-			<wheelAcceleration>${wheel_acceleration}</wheelAcceleration>
-			<commandTopic>${cmd_topic}</commandTopic>
-			<odometryTopic>${odom_topic}</odometryTopic>
-			<odometryFrame>${odom_frame}</odometryFrame>
-			<alwaysOn>${ros_plugin_always_on}</alwaysOn>
-			<updateRate>${ros_plugin_update_rate}</updateRate>
-			<odometrySource>${ros_plugin_odom_source}</odometrySource>
-			<leftJoint>${ros_plugin_controller_name}_wheel_left_joint</leftJoint>
-			<rightJoint>${ros_plugin_controller_name}_wheel_right_joint</rightJoint>
-			<rosDebugLevel>${debugLevel}</rosDebugLevel>
-			<publishWheelTF>${ros_plugin_publish_wheel_tf}</publishWheelTF>
-			<publishWheelJointState>${ros_plugin_publish_wheel_joint_state}</publishWheelJointState>
-			<publishTf>${ros_plugin_publish_tf}</publishTf>
-		</plugin>
-	</gazebo>
+	params="parent
+	wheel_base_center_x
+	wheel_separation
+	wheel_diameter
+	wheel_torque
+	wheel_acceleration
+	wheel_joint_limit_vel
+	wheel_joint_limit_effort
+	wheel_friction1
+	wheel_friction2
+	wheel_contact_damping
+	wheel_contact_stiffness
+	wheel_mass
+	wheel_width
+	z_dist
+	cmd_topic
+	odom_topic
+	odom_frame
+	ros_plugin_always_on
+	ros_plugin_controller_name
+	ros_plugin_update_rate
+	ros_plugin_odom_source
+	ros_plugin_publish_wheel_joint_state
+	ros_plugin_publish_wheel_tf
+	ros_plugin_publish_tf
+	">
+<xacro:rr_wheel_solid
+	name="${ros_plugin_controller_name}_wheel_left"
+	parent="${parent}"
+	radius="${wheel_diameter/2}"
+	width="${wheel_width}"
+	mass="${wheel_mass}"
+	origin_x="${wheel_base_center_x}"
+	origin_y="${-(wheel_separation+wheel_width)/2}"
+	origin_z="${z_dist}"
+	limit_vel="${wheel_joint_limit_vel}"
+	limit_effort="${wheel_joint_limit_effort}"
+	contact_stiffness="${wheel_contact_stiffness}"
+	contact_damping="${wheel_contact_damping}"
+	friction1="${wheel_friction1}"
+	friction2="${wheel_friction2}"
+/>
+<xacro:rr_wheel_solid
+	name="${ros_plugin_controller_name}_wheel_right"
+	parent="${parent}"
+	radius="${wheel_diameter/2}"
+	width="${wheel_width}"
+	mass="${wheel_mass}"
+	origin_x="${wheel_base_center_x}"
+	origin_y="${(wheel_separation+wheel_width)/2}"
+	origin_z="${z_dist}"
+	limit_vel="${wheel_joint_limit_vel}"
+	limit_effort="${wheel_joint_limit_effort}"
+	contact_stiffness="${wheel_contact_stiffness}"
+	contact_damping="${wheel_contact_damping}"
+	friction1="${wheel_friction1}"
+	friction2="${wheel_friction2}"
+/>
+<gazebo>
+	<plugin name="${ros_plugin_controller_name}"
+		filename="libgazebo_ros_diff_drive.so">
+		<robotBaseFrame>${parent}</robotBaseFrame>
+		<wheelSeparation>${wheel_separation}</wheelSeparation>
+		<wheelDiameter>${wheel_diameter}</wheelDiameter>
+		<wheelTorque>${wheel_torque}</wheelTorque>
+		<wheelAcceleration>${wheel_acceleration}</wheelAcceleration>
+		<commandTopic>${cmd_topic}</commandTopic>
+		<odometryTopic>${odom_topic}</odometryTopic>
+		<odometryFrame>${odom_frame}</odometryFrame>
+		<alwaysOn>${ros_plugin_always_on}</alwaysOn>
+		<updateRate>${ros_plugin_update_rate}</updateRate>
+		<odometrySource>${ros_plugin_odom_source}</odometrySource>
+		<leftJoint>${ros_plugin_controller_name}_wheel_left_joint</leftJoint>
+		<rightJoint>${ros_plugin_controller_name}_wheel_right_joint</rightJoint>
+		<rosDebugLevel>${debugLevel}</rosDebugLevel>
+		<publishWheelTF>${ros_plugin_publish_wheel_tf}</publishWheelTF>
+		<publishWheelJointState>${ros_plugin_publish_wheel_joint_state}</publishWheelJointState>
+		<publishTf>${ros_plugin_publish_tf}</publishTf>
+	</plugin>
+</gazebo>
 </xacro:macro>
 </robot>

File: defs/drive/wheel_solid.xacro (robot description, xacro)
@@ -7,5 +7,5 @@
 	<xacro:macro name="rr_wheel_solid"
 			         params="name
-						     base_frame
+						     parent
 			                 radius
 			                 width
@@ -49,5 +49,5 @@
 		<origin xyz="${origin_x} ${origin_y} ${origin_z}" py="0 0 0"/>
     	<limit effort="${limit_effort}" velocity="${limit_vel}" />
-   		<parent link="${base_frame}"/>
+   		<parent link="${parent}"/>
 		<child link="${name}"/>
 	</joint>

File: defs/sensors/distance/laser_2d.xacro (robot description, xacro)
@@ -31,4 +31,5 @@
   <gazebo reference="${name}_link">
     <sensor type="gpu_ray" name="${name}_sensor">
+      <xacro:insert_block name="laser_pose" />
       <visualize>${visualize}</visualize>
       <update_rate>${update_rate}</update_rate>
@@ -60,72 +61,3 @@
   </gazebo>
 </xacro:macro>
-<xacro:macro name="rplidar" params="id
-								topic_name
-								frame_name
-								parent_link
-								x y z roll pitch yaw
-								update_rate
-								visualize
-								">
-  <!-- RPLidar Laser -->
-  <link name="rplidar${id}_link">
-    <collision>
-      <origin xyz="0 0 ${0.098/2}" rpy="0 0 0"/>
-      <geometry>
-    	<box size="0.098 0.07 0.1" />
-      </geometry>
-    </collision>
-    <visual>
-      <origin xyz="0 0 ${0.098/2}" rpy="0 0 0"/>
-      <geometry>
-        <box size="0.098 0.07 0.1" />
-      </geometry>
-	  <material name="Black">
-		<color rgba="0 0 0 1"/>
-	  </material>
-    </visual>
-    <inertial>
-      <mass value="1e-5" />
-      <origin xyz="0 0 0" rpy="0 0 0"/>
-      <inertia ixx="1e-6" ixy="0" ixz="0" iyy="1e-6" iyz="0" izz="1e-6" />
-    </inertial>
-  </link>
-  <joint name="rplidar${id}_joint" type="fixed">
-    <axis xyz="0 1 0" />
-    <origin xyz="${x} ${y} ${z}" rpy="${roll} ${pitch} ${yaw}"/>
-    <parent link="${parent_link}"/>
-    <child link="rplidar${id}_link"/>
-  </joint>
-    <gazebo reference="rplidar${id}_link">
-    <material value="Gazebo/FlatBlack" />
-    <sensor type="gpu_ray" name="head_rplidar${id}_sensor">
-      <visualize>${visualize}</visualize>
-      <update_rate>${update_rate}</update_rate>
-      <ray>
-        <scan>
-          <horizontal>
-            <samples>360</samples>
-            <resolution>1</resolution>
-            <min_angle>0</min_angle>
-            <max_angle>${2*rr_const_pi}</max_angle>
-          </horizontal>
-        </scan>
-        <range>
-          <min>0.20</min>
-          <max>6.0</max>
-          <resolution>0.005</resolution>
-        </range>
-        <noise>
-          <type>gaussian</type>
-          <mean>0.0</mean>
-          <stddev>0.01</stddev>
-        </noise>
-      </ray>
-      <plugin name="gazebo_ros_head_rplidar${id}_controller" filename="libgazebo_ros_gpu_laser.so">
-      	<topicName>${topic_name}</topicName>
-        <frameName>rplidar${id}_link</frameName>
-      </plugin>
-    </sensor>
-  </gazebo>
-</xacro:macro>
 </robot>

File: defs/test_robots/diff_drive_bot/drive.xacro (robot description, xacro)
@@ -5,5 +5,5 @@
        xmlns:xacro="http://ros.org/wiki/xacro">
 <xacro:rr_diff_drive
-	 base_frame="base_link"
+	 parent="base_link"
 	 wheel_base_center_x="0"
      wheel_separation ="${chassis_width}"

File: defs/test_robots/diff_drive_bot/laser.xacro (robot description, xacro)
@@ -7,6 +7,6 @@
 	name="laser"
 	topic_name="scan/laser"
-	update_rate="5.5"
-	visualize="false"
+	update_rate="10"
+	visualize="true"
 	hor_samples="360"
 	hor_resolution="1"
@@ -17,5 +17,5 @@
 	range_resolution="0.005"
 	noise_type="gaussian"
-    noise_mean="0.0"
+    noise_mean="0.01"
     noise_stddev="0.01"
 	parent="base_link"
