Commit message: fix imu and gps to have included tags

File: defs/sensors/contact/bumper.xacro (robot description, xacro)
@@ -29,5 +29,5 @@
 -->
 <xacro:macro name="rr_bumper"
-	params="name parent has_inertia always_on update_rate topic *origin *geometry *material *inertial">
+	params="name parent always_on update_rate topic has_inertia *origin *geometry *material *inertial">
 	<link name="${name}">
 	  <visual>

File: defs/sensors/inertia/imu.xacro (robot description, xacro)
@@ -7,23 +7,4 @@
 <!-- Example -->
 <!--
-<xacro:rr_imu
-		name="imu0"
-	 	robot_namespace=""
-		topic_name="/imu"
-		parent_link="chassis"
-		x="${wheel_base_center_x}"
-		y="0"
-		z="0"
-		roll="0"
-		pitch="0"
-		yaw="0"
-		gaussian_noise="2.89e-08"
-		imu_x="0"
-		imu_y="0"
-		imu_z="0"
-		imu_roll="0"
-		imu_pitch="0"
-		imu_yaw="0"
-		/>
 -->
 <xacro:macro name="rr_imu" params="name
@@ -31,22 +12,33 @@
 								topic_name
 								parent_link
-								x y z roll pitch yaw
 								gaussian_noise
-								imu_x imu_y imu_z imu_roll imu_pitch imu_yaw
+								imu_x
+								imu_y
+								imu_z
+								imu_roll
+								imu_pitch
+								imu_yaw
+	                            has_inertia
+							    *origin
+							    *geometry
+							    *material
+							    *inertial
 								">
 <link name="${name}_link">
-	<visual>
-		<geometry>
-			<box size="0.02 0.02 0.02" />
-		</geometry>
-		<material name="Yellow">
-			<color rgba="1 1 0 1"/>
-		</material>
-	</visual>
+  <visual>
+      <xacro:insert_block name="geometry" />
+	  <xacro:insert_block name="material" />
+  </visual>
+  <collision name="${name}_collision">
+  	  	<xacro:insert_block name="geometry" />
+  </collision>
+  <xacro:if value="${has_inertia}">
+	<xacro:insert_block name="inertial" />
+  </xacro:if>
 </link>
 <joint name="${name}_joint" type="fixed">
 	<parent link="${parent_link}" />
 	<child link="${name}_link" />
-	<origin xyz="${x} ${y} ${z}" rpy="${roll} ${pitch} ${yaw}" />
+	<xacro:insert_block name="origin" />
 </joint>
 <gazebo>
@@ -56,6 +48,6 @@
 			<topicName>${topic_name}</topicName>
 			<gaussianNoise>${gaussian_noise}</gaussianNoise>
-			<xyzOffsets>0 0 0</xyzOffsets>
-			<rpyOffsets>0 0 0</rpyOffsets>
+			<xyzOffsets>${imu_x} ${imu_y} ${imu_z}</xyzOffsets>
+			<rpyOffsets>${imu_roll} ${imu_pitch} ${imu_yaw}</rpyOffsets>
 	  </plugin>
 </gazebo>

File: defs/sensors/position/gps.xacro (robot description, xacro)
@@ -10,6 +10,5 @@
 		name="gps0"
 	 	robot_namespace="${robot_namespace}"
-		parent_link="chassis"
-		x="0" y="0" z="0"
+		parent_link="base_link"
 		frame_id="world"
 		topic_name="/fix"
@@ -18,5 +17,20 @@
 		reference_longitude="8"
 		reference_heading="0"
-		reference_altitude="0"/>
+		reference_altitude="0"
+		has_inertia="true">
+	    <origin xyz="0 0 0" rpy="0 0 0" />
+		<geometry>
+			<box size="0.04 0.03 0.02" />
+		</geometry>
+		<material name="Black">
+			<color rgba="0 0 0 1"/>
+		</material>
+		 <xacro:inertia_box x="0.02" y="0.02" z="0.04" mass="0.1">
+	      <origin xyz="0 0 0" rpy="0 0 0" />
+	    </xacro:inertia_box>
+	</xacro:rr_gps_receiver>
+	<gazebo reference="gps0">
+		<material value="Gazebo/FlatBlack" />
+	</gazebo>
 -->
 <xacro:macro name="rr_gps_receiver"
@@ -26,5 +40,4 @@
 		 topic_name
 		 parent_link
-		 x y z
 		 velocity_topic_name
 		 reference_latitude
@@ -32,25 +45,32 @@
 		 reference_heading
 		 reference_altitude
+	     has_inertia
+	     *origin
+	     *geometry
+	     *material
+	     *inertial
 		">
-	<link name="${name}_receiver_link">
-		<visual>
-			<geometry>
-				<box size="0.04 0.04 0.04" />
-			</geometry>
-			<material name="Blue">
-				<color rgba="0 0 1 1"/>
-			</material>
-		</visual>
-	</link>
-	<joint name="${name}_receiver_joint" type="fixed">
-		<parent link="${parent_link}" />
-		<child link="${name}_receiver_link" />
-		<origin xyz="${x} ${y} ${z}" rpy="0 0 0" />
-	</joint>
+<link name="${name}_link">
+  <visual>
+      <xacro:insert_block name="geometry" />
+	  <xacro:insert_block name="material" />
+  </visual>
+  <collision name="${name}_collision">
+  	  	<xacro:insert_block name="geometry" />
+  </collision>
+  <xacro:if value="${has_inertia}">
+	<xacro:insert_block name="inertial" />
+  </xacro:if>
+</link>
+<joint name="${name}_joint" type="fixed">
+	<parent link="${parent_link}" />
+	<child link="${name}_link" />
+	<xacro:insert_block name="origin" />
+</joint>
 <gazebo>
 	<plugin name="${name}_controller"
 		    filename="libhector_gazebo_ros_gps.so">
 		<robotNamespace>${robot_namespace}</robotNamespace>
-		<bodyName>${name}_receiver_link</bodyName>
+		<bodyName>${name}_link</bodyName>
 		<frameId>${frame_id}</frameId>
 		<topicName>${topic_name}</topicName>

File: defs/test_robots/diff_drive_bot.xacro (robot description, xacro)
@@ -15,10 +15,12 @@
 <xacro:property name="caster_collision_x"      value="${chassis_len/(1.618*2)}"        />
 <xacro:property name="robot_namespace" value="/" />
+<xacro:property name="chassis_center" value="${chassis_floor_clearance+chassis_height/2}" />
 <!--CHASSIS-->
-<link name="chassis">
-	 <xacro:rr_inertia_box_solid x="${chassis_len}" y="${chassis_width}" z="${chassis_height}" mass="1">
-      <origin xyz="0 0 ${chassis_floor_clearance}" rpy="0 0 0" />
+<link name="base_link">
+	<xacro:rr_inertia_box_solid x="${chassis_len}" y="${chassis_width}" z="${chassis_height}" mass="1">
+      	 <origin xyz="0 0 ${chassis_center}" rpy="0 0 0" />
     </xacro:rr_inertia_box_solid>
 	<visual>
+		<origin xyz="0 0 ${chassis_center}" rpy="0 0 0" />
 		<geometry>
 			<box size="${chassis_len} ${chassis_width} ${chassis_height}" />
@@ -29,4 +31,5 @@
 	</visual>
 	<collision>
+		<origin xyz="0 0 ${chassis_center}" rpy="0 0 0" />
 		<geometry>
 			<box size="${chassis_len} ${chassis_width} ${chassis_height}" />
@@ -34,10 +37,10 @@
 	</collision>
 </link>
-<gazebo reference="chassis">
+<gazebo reference="base_link">
 	<material value="Gazebo/Green"/>
 </gazebo>
 <!-- Bumper -->
-<xacro:rr_bumper name="bumper0" parent="chassis" always_on="true" update_rate="30" topic="bumper0"  has_inertia="true">
-	<origin xyz="${chassis_len/2} ${chassis_width/2} 0" rpy="0 0 0" />
+<xacro:rr_bumper name="bumper0" parent="base_link" always_on="true" update_rate="30" topic="bumper0"  has_inertia="true">
+	<origin xyz="${chassis_len/2} ${chassis_width/2} ${chassis_center}" rpy="0 0 0" />
 	<geometry>
 		<box size="0.02 0.02 ${chassis_height}" />
@@ -53,6 +56,6 @@
 	<material value="Gazebo/FlatBlack" />
 </gazebo>
-<xacro:rr_bumper name="bumper1" parent="chassis" always_on="true" update_rate="30" topic="bumper1"  has_inertia="true">
-	<origin xyz="${chassis_len/2} -${chassis_width/2} 0" rpy="0 0 0" />
+<xacro:rr_bumper name="bumper1" parent="base_link" always_on="true" update_rate="30" topic="bumper1"  has_inertia="true">
+	<origin xyz="${chassis_len/2} -${chassis_width/2} ${chassis_center}" rpy="0 0 0" />
 	<geometry>
 		<box size="0.02 0.02 ${chassis_height}" />
@@ -68,6 +71,6 @@
 	<material value="Gazebo/FlatBlack" />
 </gazebo>
-<xacro:rr_bumper name="bumper2" parent="chassis" always_on="true" update_rate="30" topic="bumper2"  has_inertia="true">
-	<origin xyz="${chassis_len/2} 0 -${chassis_height/4}" rpy="0 0 0" />
+<xacro:rr_bumper name="bumper2" parent="base_link" always_on="true" update_rate="30" topic="bumper2"  has_inertia="true">
+	<origin xyz="${chassis_len/2} 0 ${chassis_center-chassis_height/4}" rpy="0 0 0" />
 	<geometry>
 		<box size="0.02 ${chassis_width-0.04} 0.02" />
@@ -113,11 +116,11 @@
 </gazebo>
 <joint name="base_caster_col_joint" type="fixed">
-	<parent link="chassis" />
+	<parent link="base_link" />
 	<child link="caster_collision" />
-	<origin xyz="${caster_collision_x} 0 ${-(chassis_height/2)}" rpy="0 0 0" />
+	<origin xyz="${caster_collision_x} 0 ${chassis_center-(chassis_height/2)}" rpy="0 0 0" />
 </joint>
 <!-- Drive -->
 <xacro:rr_diff_drive
-	 base_frame="chassis"
+	 base_frame="base_link"
 	 robot_namespace="${robot_namespace}"
 	 wheel_base_center_x="${wheel_base_center_x}"
@@ -134,5 +137,5 @@
      wheel_contact_stiffness="1000000.0"
 	 wheel_mass="3"
-	 z_dist="${-((chassis_floor_clearance+chassis_height/2)-(wheel_diameter/2))}"
+	 z_dist="${chassis_center-((chassis_floor_clearance+chassis_height/2)-(wheel_diameter/2))}"
      cmd_topic="/cmd_vel"
 	 odom_topic="odom"
@@ -145,3 +148,104 @@
 	 ros_plugin_publish_wheel_tf="true"
 	 ros_plugin_publish_tf="1" />
+<!-- GPS -->
+	<xacro:rr_gps_receiver
+		name="gps0"
+	 	robot_namespace="${robot_namespace}"
+		parent_link="base_link"
+		frame_id="world"
+		topic_name="/fix"
+		velocity_topic_name="/fix_vel"
+		reference_latitude="49"
+		reference_longitude="8"
+		reference_heading="0"
+		reference_altitude="0"
+		has_inertia="true">
+	    <origin xyz="${-(chassis_len/2-0.04/2)} ${chassis_width/2-0.015}
+                     ${chassis_center+chassis_height/2+0.02/2}"
+	                 rpy="0 0 0" />
+		<geometry>
+			<box size="0.04 0.03 0.02" />
+		</geometry>
+		<material name="Black">
+			<color rgba="0 0 0 1"/>
+		</material>
+		 <xacro:inertia_box x="0.02" y="0.02" z="0.04" mass="0.1">
+	      <origin xyz="0 0 0" rpy="0 0 0" />
+	    </xacro:inertia_box>
+	</xacro:rr_gps_receiver>
+	<gazebo reference="gps0">
+		<material value="Gazebo/FlatBlack" />
+	</gazebo>
+<!-- IMU -->
+<xacro:rr_imu
+		name="imu0"
+	 	robot_namespace=""
+		topic_name="/imu"
+		parent_link="base_link"
+		gaussian_noise="2.89e-08"
+		imu_x="0"
+		imu_y="0"
+		imu_z="0"
+		imu_roll="0"
+		imu_pitch="0"
+		imu_yaw="0"
+		has_inertia="false"
+		>
+		<origin xyz="${wheel_base_center_x}
+                       0
+		             ${chassis_center-((chassis_floor_clearance+
+                       chassis_height/2)-(wheel_diameter/2))}" rpy="0 0 0" />
+		<geometry>
+			<box size="0.02 0.02 0.02" />
+		</geometry>
+		<material name="Yellow">
+			<color rgba="1 1 0 1"/>
+		</material>
+		 <inertial/>
+	</xacro:rr_imu>
+<!-- CAMERA
+<xacro:rr_cam
+		name             ="cam0"
+	 	robot_namespace  ="${robot_namespace}"
+		parent_link      ="base_link"
+		x                ="${chassis_len/2}"
+	    y                ="0"
+        z                ="0"
+        roll             ="0"
+        pitch            ="-0.01"
+        yaw              ="0"
+		always_on        ="true"
+		frame_name       ="camera0"
+		image_width      ="640"
+		image_height     ="480"
+		image_format     ="R8G8B8"
+		clip_near        ="0.02"
+		clip_far         ="300"
+		noise_type       ="gaussian"
+		noise_mean       ="0.0"
+		noise_std_dev    ="0.007"
+		fov              ="0.873"
+		hack_baseline    ="0.07"
+		dist_K1          ="0.0"
+		dist_K2          ="0.0"
+		dist_K3          ="0.0"
+		dist_T1          ="0.0"
+		dist_T2          ="0.0"
+		update_rate      ="30"
+        />	 -->
+<!-- LIDAR
+<xacro:rplidar id="0"
+	 	robot_namespace="${robot_namespace}"
+		topic_name="/laser/scan"
+		frame_name="laser"
+		parent_link="base_link"
+		x="0"
+        y="0"
+        z="${chassis_height/2}"
+	    roll="0"
+	    pitch="0"
+        yaw="0"
+		update_rate="5.5"
+		visualize="false" />
+ -->
 </robot>

Commit message: remove examples - use the ones from the test robot

File: defs/sensors/contact/bumper.xacro (robot description, xacro)
@@ -4,28 +4,4 @@
        xmlns:interface="http://playerstage.sourceforge.net/gazebo/xmlschema/#interface"
        xmlns:xacro="http://ros.org/wiki/xacro">
-<!-- Example
-	Inertial tags must be there but they can be empty when has_inertia is false
- -->
-<!--
-<xacro:rr_bumper name="bumper0"
-              parent="chassis"
-              always_on="true"
-              update_rate="30"
-	          topic="bumper0"
-              has_inertia="false">
-	<origin xyz="${chassis_len/2} ${chassis_width/2} 0" rpy="0 0 0" />
-	<geometry>
-		<box size="0.1 0.1 0.1" />
-	</geometry>
-	<material name="Green">
-		<color rgba="0 1 0 0.5"/>
-	</material>
-	<inertial>
-	</inertial>
-</xacro:bumper>
-<gazebo reference="bumper0">
-	<material value="Gazebo/FlatBlack" />
-</gazebo>
--->
 <xacro:macro name="rr_bumper"
 	params="name parent always_on update_rate topic has_inertia *origin *geometry *material *inertial">

File: defs/sensors/imaging/camera.xacro (robot description, xacro)
@@ -5,42 +5,4 @@
        xmlns:xacro="http://ros.org/wiki/xacro">
 <xacro:include filename="$(find rapid_robot_xacros)/defs/geometry/geo_ins.xacro"/>
-<!-- Example -->
-<!--
-<xacro:rr_cam
-	name             ="cam0"
-	always_on        ="true"
-	frame_name       ="camera0"
-	image_width      ="640"
-	image_height     ="480"
-	image_format     ="R8G8B8"
-	clip_near        ="0.02"
-	clip_far         ="300"
-	noise_type       ="gaussian"
-	noise_mean       ="0.0"
-	noise_std_dev    ="0.007"
-	fov              ="0.873"
-	hack_baseline    ="0.07"
-	dist_K1          ="0.0"
-	dist_K2          ="0.0"
-	dist_K3          ="0.0"
-	dist_T1          ="0.0"
-	dist_T2          ="0.0"
-	update_rate      ="30"
-	parent           ="base_link"
-    has_inertia      ="false"
-	>
-	<origin xyz="${chassis_len/2}
-                 0
-	             ${chassis_center}" rpy="0 0 0" />
-	<geometry>
-		<box size="0.02 0.02 0.02" />
-	</geometry>
-	<material name="Yellow">
-		<color rgba="0 0 0 1"/>
-	</material>
-	 <inertial/>
-    </xacro:rr_cam>
-	<xacro:rr_gaz_mat_s name="cam0" material="Gazebo/FlatBlack"/>
--->
 <xacro:macro name="rr_cam"
 	params="

File: defs/sensors/inertia/imu.xacro (robot description, xacro)
@@ -6,33 +6,4 @@
 >
 <xacro:include filename="$(find rapid_robot_xacros)/defs/geometry/geo_ins.xacro"/>
-<!-- Example -->
-<!--
-<xacro:rr_imu
-	name="imu0"
- 	robot_namespace=""
-	topic_name="/imu"
-	gaussian_noise="2.89e-08"
-	imu_x="0"
-	imu_y="0"
-	imu_z="0"
-	imu_roll="0"
-	imu_pitch="0"
-	imu_yaw="0"
-	parent="base_link"
-	has_inertia="false"
-	>
-	<origin xyz="${wheel_base_center_x}
-                   0
-	             ${chassis_center-((chassis_floor_clearance+
-                   chassis_height/2)-(wheel_diameter/2))}" rpy="0 0 0" />
-	<geometry>
-		<box size="0.02 0.02 0.02" />
-	</geometry>
-	<material name="Yellow">
-		<color rgba="1 1 0 1"/>
-	</material>
-	 <inertial/>
-</xacro:rr_imu>
--->
 <xacro:macro name="rr_imu" params="name
 								topic_name

File: defs/sensors/position/gps.xacro (robot description, xacro)
@@ -6,32 +6,4 @@
 >
 <xacro:include filename="$(find rapid_robot_xacros)/defs/geometry/geo_ins.xacro"/>
-<!-- Example -->
-<!--
-	<xacro:rr_gps_receiver
-		name="gps0"
-		frame_id="world"
-		topic_name="/fix"
-		velocity_topic_name="/fix_vel"
-		reference_latitude="49"
-		reference_longitude="8"
-		reference_heading="0"
-		reference_altitude="0"
-		parent="base_link"
-		has_inertia="true">
-	    <origin xyz="0 0 0" rpy="0 0 0" />
-		<geometry>
-			<box size="0.04 0.03 0.02" />
-		</geometry>
-		<material name="Black">
-			<color rgba="0 0 0 1"/>
-		</material>
-		 <xacro:inertia_box x="0.02" y="0.02" z="0.04" mass="0.1">
-	      <origin xyz="0 0 0" rpy="0 0 0" />
-	    </xacro:inertia_box>
-	</xacro:rr_gps_receiver>
-	<gazebo reference="gps0">
-		<material value="Gazebo/FlatBlack" />
-	</gazebo>
--->
 <xacro:macro name="rr_gps_receiver"
 params= "name

Commit message: formatting code

File: defs/sensors/contact/bumper.xacro (robot description, xacro)
@@ -5,5 +5,14 @@
        xmlns:xacro="http://ros.org/wiki/xacro">
 <xacro:macro name="rr_bumper"
-	params="name parent always_on update_rate topic has_inertia *origin *geometry *material *inertial">
+	params="name
+			parent
+			always_on
+			update_rate
+			topic
+			has_inertia
+			*origin
+			*geometry
+			*material
+			*inertial">
 	<xacro:rr_geo_ins/>
 	<gazebo reference="${name}_link">

File: defs/test_robots/diff_drive_bot/bumpers.xacro (robot description, xacro)
@@ -4,36 +4,46 @@
        xmlns:interface="http://playerstage.sourceforge.net/gazebo/xmlschema/#interface"
        xmlns:xacro="http://ros.org/wiki/xacro">
-<xacro:rr_bumper name="bumper0" parent="base_link" always_on="true"
-       	       update_rate="30" topic="bumper0"  has_inertia="true">
-	<origin xyz="${chassis_len/2-wheel_base_center_x} ${chassis_width/2} ${chassis_center_z}" rpy="0 0 0" />
+<xacro:rr_bumper name="bumper0" parent="base_link" always_on="true" update_rate="30"
+	topic="bumper0" has_inertia="true">
+	<origin xyz="${chassis_len/2-wheel_base_center_x}
+	             ${chassis_width/2}
+		         ${chassis_center_z}"
+		    rpy="0 0 0" />
 	<geometry>
 		<box size="0.02 0.02 ${chassis_height}" />
 	</geometry>
 	<material name="rr_m_black"/>
-	 <xacro:rr_inertia_box_solid x="0.02" y="0.02" z="${chassis_height}" mass="0.1">
-      <origin xyz="0 0 0" rpy="0 0 0" />
-    </xacro:rr_inertia_box_solid>
+	<xacro:rr_inertia_box_solid x="0.02" y="0.02" z="${chassis_height}" mass="0.1">
+		<origin xyz="0 0 0" rpy="0 0 0" />
+	</xacro:rr_inertia_box_solid>
 </xacro:rr_bumper>
 <xacro:rr_m_gz_black name="bumper0"/>
-<xacro:rr_bumper name="bumper1" parent="base_link" always_on="true" update_rate="30" topic="bumper1"  has_inertia="true">
-	<origin xyz="${chassis_len/2-wheel_base_center_x} -${chassis_width/2} ${chassis_center_z}" rpy="0 0 0" />
+<xacro:rr_bumper name="bumper1" parent="base_link" always_on="true" update_rate="30"
+	topic="bumper1" has_inertia="true">
+	<origin xyz="${chassis_len/2-wheel_base_center_x} -${chassis_width/2} ${chassis_center_z}"
+		rpy="0 0 0" />
 	<geometry>
 		<box size="0.02 0.02 ${chassis_height}" />
 	</geometry>
 	<material name="rr_m_black"/>
-	 <xacro:inertia_box x="0.02" y="0.02" z="${chassis_height}" mass="0.1">
-      <origin xyz="0 0 0" rpy="0 0 0" />
-    </xacro:inertia_box>
+	<xacro:inertia_box x="0.02" y="0.02" z="${chassis_height}" mass="0.1">
+		<origin xyz="0 0 0" rpy="0 0 0" />
+	</xacro:inertia_box>
 </xacro:rr_bumper>
 <xacro:rr_m_gz_black name="bumper1"/>
-<xacro:rr_bumper name="bumper2" parent="base_link" always_on="true" update_rate="30" topic="bumper2"  has_inertia="true">
-	<origin xyz="${chassis_len/2-wheel_base_center_x} 0 ${chassis_center_z-chassis_height/4}" rpy="0 0 0" />
+<xacro:rr_bumper name="bumper2" parent="base_link"
+	             always_on="true" update_rate="30"
+	             topic="bumper2" has_inertia="true">
+	<origin xyz="${chassis_len/2-wheel_base_center_x}
+				 0
+	             ${chassis_center_z-chassis_height/4}"
+		    rpy="0 0 0" />
 	<geometry>
 		<box size="0.02 ${chassis_width-0.04} 0.02" />
 	</geometry>
 	<material name="rr_m_black"/>
-	 <xacro:inertia_box x="0.02" y="0.02" z="0.04" mass="0.1">
-      <origin xyz="0 0 0" rpy="0 0 0" />
-    </xacro:inertia_box>
+	<xacro:inertia_box x="0.02" y="0.02" z="0.04" mass="0.1">
+		<origin xyz="0 0 0" rpy="0 0 0" />
+	</xacro:inertia_box>
 </xacro:rr_bumper>
 <xacro:rr_m_gz_black name="bumper2"/>

File: defs/test_robots/diff_drive_bot/drive.xacro (robot description, xacro)
@@ -19,5 +19,8 @@
 	wheel_contact_stiffness="1000000.0"
 	wheel_mass="1"
-	z_dist="${chassis_center_z-((chassis_floor_clearance+chassis_height/2)-(wheel_diameter/2))}"
+	z_dist="${chassis_center_z-
+              ((chassis_floor_clearance
+               +chassis_height/2)
+               -(wheel_diameter/2))}"
 	cmd_topic="cmd_vel"
 	odom_topic="odom"

File: defs/test_robots/diff_drive_bot/imu.xacro (robot description, xacro)
@@ -18,6 +18,7 @@
 		>
 		<origin xyz="0 0
-		             ${chassis_center_z-((chassis_floor_clearance+
-                       chassis_height/2)-(wheel_diameter/2))}" rpy="0 0 0" />
+		        ${chassis_center_z-((chassis_floor_clearance+
+                chassis_height/2)-(wheel_diameter/2))}"
+		        rpy="0 0 0" />
 		<geometry>
 			<box size="0.02 0.02 0.02" />
