Commit message: add another value for wheel separation

File: def/drive/diff_drive.xacro (robot description, xacro)
@@ -69,6 +69,6 @@
 		filename="libgazebo_ros_diff_drive.so">
 		<robotBaseFrame>${parent}</robotBaseFrame>
-		<wheelSeparation>${wheel_separation+wheel_width}</wheelSeparation>
-		<wheelDiameter>${wheel_diameter/2}</wheelDiameter>
+		<wheelSeparation>${(wheel_separation+wheel_width)*2}</wheelSeparation>
+		<wheelDiameter>${wheel_diameter}</wheelDiameter>
 		<wheelTorque>${wheel_torque}</wheelTorque>
 		<wheelAcceleration>${wheel_acceleration}</wheelAcceleration>

File: def/test_robots/diff_drive_bot/drive.xacro (robot description, xacro)
@@ -7,5 +7,5 @@
 	parent="base_link"
 	wheel_base_center_x="0"
-	wheel_separation ="${chassis_width}"
+	wheel_separation ="${wheel_separation}"
 	wheel_diameter="${wheel_diameter}"
 	wheel_width="${wheel_width}"

File: def/test_robots/diff_drive_bot/properties.xacro (robot description, xacro)
@@ -15,3 +15,5 @@
 <xacro:property name="chassis_center_z"
 				value="${chassis_floor_clearance+chassis_height/2}" />
+<xacro:property name="wheel_separation"
+                value="0.38" />
 </robot>
