Commit message: add changes and fix wheels

File: def/test_robots/diff_drive_bot/drive.xacro (robot description, xacro)
@@ -5,31 +5,28 @@
        xmlns:xacro="http://ros.org/wiki/xacro">
 <xacro:rr_diff_drive
-	parent="base_link"
-	wheel_base_center_x="0"
-	wheel_separation ="${wheel_separation}"
-	wheel_diameter="${wheel_diameter}"
-	wheel_width="${wheel_width}"
-	wheel_torque="5"
-	wheel_acceleration="1"
-	wheel_joint_limit_vel="2"
-	wheel_joint_limit_effort="2"
-	wheel_friction1="100000"
-	wheel_friction2="1000"
-	wheel_contact_damping="100.0"
-	wheel_contact_stiffness="1000000.0"
-	wheel_mass="0.5"
-	z_dist="${chassis_center_z-
-              ((chassis_floor_clearance
-               +chassis_height/2)
-               -(wheel_diameter/2))}"
-	cmd_topic="cmd_vel"
-	odom_topic="odom"
-	odom_frame="odom"
-	ros_plugin_always_on="true"
-	ros_plugin_controller_name="diff_drv0"
-	ros_plugin_update_rate="100"
-	ros_plugin_odom_source="encoder"
-	ros_plugin_publish_wheel_joint_state="true"
-	ros_plugin_publish_wheel_tf="true"
-	ros_plugin_publish_tf="1" />
+     parent="base_link"
+     wheel_base_center_x="0"
+     wheel_separation ="${wheel_separation}"
+     wheel_diameter="${wheel_diameter}"
+     wheel_width="${wheel_width}"
+     wheel_torque="5.0"
+     wheel_acceleration="1.0"
+     wheel_joint_limit_vel="2.0"
+     wheel_joint_limit_effort="2.0"
+     wheel_friction1="100.0"
+     wheel_friction2="100.0"
+     wheel_contact_damping="1.0"
+     wheel_contact_stiffness="1000000.0"
+     wheel_mass="0.513"
+     z_dist="0.12"
+     cmd_topic="/cmd_vel"
+     odom_topic="odom"
+     odom_frame="odom"
+     ros_plugin_always_on="true"
+     ros_plugin_controller_name="diff_drv0"
+     ros_plugin_update_rate="30"
+     ros_plugin_odom_source="world"
+     ros_plugin_publish_wheel_joint_state="true"
+     ros_plugin_publish_wheel_tf="true"
+     ros_plugin_publish_tf="1" />
 </robot>

File: def/test_robots/diff_drive_bot/gps.xacro (robot description, xacro)
@@ -4,13 +4,11 @@
        xmlns:interface="http://playerstage.sourceforge.net/gazebo/xmlschema/#interface"
        xmlns:xacro="http://ros.org/wiki/xacro">
-<xacro:rr_gps_receiver
+<xacro:rr_gps_hector
 	name="gps0"
-	frame_id="world"
-	topic_name="fix"
-	velocity_topic_name="fix_vel"
-	reference_latitude="49"
-	reference_longitude="8"
+	topic_name="/gps/fix"
+	reference_latitude="48.652726006"
+	reference_longitude="9.184366555"
 	reference_heading="0"
-	reference_altitude="0"
+	reference_altitude="472.05"
 	parent="base_link"
 	has_inertia="true">
@@ -24,8 +22,8 @@
 		<color rgba="0 0 0 1"/>
 	</material>
-	 <xacro:inertia_box x="0.02" y="0.02" z="0.04" mass="0.1">
+	 <!--xacro:inertia_box x="0.02" y="0.02" z="0.04" mass="0.1">
       <origin xyz="0 0 0" rpy="0 0 0" />
-    </xacro:inertia_box>
-</xacro:rr_gps_receiver>
-<xacro:rr_gaz_mat_s name="gps0" material="Gazebo/FlatBlack"/>
+    </xacro:inertia_box-->
+</xacro:rr_gps_hector>
+<xacro:rr_m_gz_black name="gps0"/>
 </robot>

File: def/test_robots/diff_drive_bot/imu.xacro (robot description, xacro)
@@ -6,6 +6,6 @@
 <xacro:rr_imu_hector
 		name="imu0"
-		topic_name="imu"
-		gaussian_noise="2.89e-08"
+		topic_name="/imu"
+		gaussian_noise="0"
 		imu_x="0"
 		imu_y="0"
@@ -13,12 +13,10 @@
 		imu_roll="0"
 		imu_pitch="0"
-		imu_yaw="${rr_const_pi*2}"
+		imu_yaw="0"
 		parent="base_link"
 		has_inertia="false"
 		>
-		<origin xyz="0 0
-		        ${chassis_center_z-((chassis_floor_clearance+
-                chassis_height/2)-(wheel_diameter/2))}"
-		        rpy="0 0 0" />
+		<!--origin xyz="0.29 0.16 ${0.5*wheel_diameter}" rpy="${-rr_const_pi/2} ${-rr_const_pi/2} ${-rr_const_pi}" /-->
+		<origin xyz="0.41 0.0 0.2" rpy="0.0 0.0 0" />
 		<geometry>
 			<box size="0.02 0.02 0.02" />
@@ -29,4 +27,4 @@
 		 <inertial/>
 	</xacro:rr_imu_hector>
-	<xacro:rr_gaz_mat_s name="imu0" material="Gazebo/Yellow"/>
+<xacro:rr_m_gz_black name="imu0"/>
 </robot>

File: def/test_robots/diff_drive_bot/laser.xacro (robot description, xacro)
@@ -5,22 +5,22 @@
        xmlns:xacro="http://ros.org/wiki/xacro">
 <xacro:rr_laser_2d
-	name="laser"
-	topic_name="scan/laser"
-	update_rate="10"
-	visualize="false"
-	hor_samples="360"
-	hor_resolution="1"
-	hor_min_angle="${0}"
-	hor_max_angle="${2*rr_const_pi}"
-	range_min="0.20"
-	range_max="6"
-	range_resolution="0.005"
-	noise_type="gaussian"
-    noise_mean="0.01"
+    name="laser"
+    topic_name="xmos_com/scan"
+    update_rate="2.0"
+    visualize="false"
+    hor_samples="360"
+    hor_resolution="1"
+    hor_min_angle="${-rr_const_pi}"
+    hor_max_angle="${rr_const_pi}"
+    range_min="0.20"
+    range_max="14"
+    range_resolution="0.005"
+    noise_type="gaussian"
+    noise_mean="0.0"
     noise_stddev="0.01"
-	parent="base_link"
+    parent="base_link"
     has_inertia="false"
 	>
-	<origin xyz="0 0 ${chassis_center_z+chassis_height/2+0.1/2}" rpy="0 0 0" />
+	<origin xyz="0 0 ${chassis_center_z+0.15}" rpy="0 0 0" />
 	<geometry>
 		<box size="0.098 0.07 0.1" />

File: def/test_robots/diff_drive_bot/properties.xacro (robot description, xacro)
@@ -4,16 +4,15 @@
        xmlns:interface="http://playerstage.sourceforge.net/gazebo/xmlschema/#interface"
        xmlns:xacro="http://ros.org/wiki/xacro">
-<xacro:property name="chassis_height" value="0.25" />
-<xacro:property name="chassis_width" value="${chassis_height*1.618}" />
-<xacro:property name="chassis_len" value="${chassis_width+chassis_height}" />
+<xacro:property name="chassis_height" value="0.18" />
+<xacro:property name="chassis_width" value="0.36" />
+<xacro:property name="chassis_len" value="0.56" />
 <xacro:property name="chassis_floor_clearance"
-				value="${chassis_height/(1.618*2)}" />
-<xacro:property name="wheel_diameter" value="${chassis_len/(1.618*1.618)}" />
-<xacro:property name="wheel_width" value="${chassis_width/(16.18)}" />
-<xacro:property name="wheel_base_center_x" value="${chassis_len/(-1.618*3)}" />
-<xacro:property name="caster_x" value="${chassis_len/(1.618*2)}"/>
+				value="0.07" />
+<xacro:property name="wheel_diameter" value="0.23" />
+<xacro:property name="wheel_width" value="0.04" />
+<xacro:property name="wheel_base_center_x" value="-0.16" />
+<xacro:property name="caster_x" value="0.21"/>
 <xacro:property name="chassis_center_z"
 				value="${chassis_floor_clearance+chassis_height/2}" />
-<xacro:property name="wheel_separation"
-                value="0.38" />
+<xacro:property name="wheel_separation" value="0.38" />
 </robot>
