Commit message: fix camera frame

File: def/sensors/imaging/camera.xacro (robot description, xacro)
@@ -71,4 +71,10 @@
 	</sensor>
 </gazebo>
+<joint name="${frame_name}_${name}_joint" type="fixed">
+	<parent link="${name}_link" />
+	<child link="${frame_name}" />
+    <origin xyz="0 0 0" rpy="-1.57 0 -1.57" />
+</joint>
+<link name="${frame_name}" ></link>
 </xacro:macro>
 </robot>
