Commit message: fix start

File: def/test_robots/portalbot.xacro (robot description, xacro)
@@ -5,4 +5,4 @@
 <xacro:include filename="$(find h4r_rapid_robot_xacros)/def/rapid_robot.xacro"/>
 <xacro:include filename="$(find h4r_rapid_robot_xacros)/def/test_robots/portalbot/properties.xacro"/>
-<xacro:include filename="$(find h4r_rapid_robot_xacros)/def/test_robots/portalbot/axis_placement.xacro"/>
+<xacro:include filename="$(find h4r_rapid_robot_xacros)/def/test_robots/portalbot/base.xacro"/>
 </robot>

File: def/test_robots/portalbot/properties.xacro (robot description, xacro)
@@ -9,4 +9,5 @@
 <xacro:property name="y_track_width"  value="${x_track_height}" />
 <xacro:property name="y_track_height" value="${x_track_width}" />
+<xacro:property name="y_bar_weight" value="1.5" />
 <xacro:property name="z_track_width"  value="${y_track_width}" />
 <xacro:property name="z_track_height" value="${x_track_height}" />

Commit message: add bar weights and axis length as parameter

File: def/test_robots/portalbot.xacro (robot description, xacro)
@@ -4,4 +4,5 @@
        xmlns:xacro="http://ros.org/wiki/xacro" name="diff_drive_bot">
 <xacro:include filename="$(find h4r_rapid_robot_xacros)/def/rapid_robot.xacro"/>
+<xacro:include filename="$(find h4r_rapid_robot_xacros)/def/test_robots/portalbot/bar.xacro"/>
 <xacro:include filename="$(find h4r_rapid_robot_xacros)/def/test_robots/portalbot/properties.xacro"/>
 <xacro:include filename="$(find h4r_rapid_robot_xacros)/def/test_robots/portalbot/base.xacro"/>

File: def/test_robots/portalbot/base.xacro (robot description, xacro)
@@ -21,6 +21,6 @@
 </link>
 </xacro:macro>
-<xacro:rr_port_base_y_side name="y_track_left"  width="${y_track_width}" len="${y_axis_len}" height="${y_track_height}" weight="${y_bar_weight}" />
-<xacro:rr_port_base_y_side name="y_track_right" width="${y_track_width}" len="${y_axis_len}" height="${y_track_height}" weight="${y_bar_weight}" />
+<xacro:rr_portal_bar name="y_track_left"  width="${y_track_width}" len="${y_axis_len}" height="${y_track_height}" weight="${y_bar_weight}" />
+<xacro:rr_portal_bar name="y_track_right" width="${y_track_width}" len="${y_axis_len}" height="${y_track_height}" weight="${y_bar_weight}" />
 <joint name="joint_y_track_right_left" type="fixed">
 	<parent link="y_track_left" />
@@ -28,6 +28,6 @@
 	<origin xyz="${x_axis_len + y_track_width} 0 0" rpy="0 0 0" />
 </joint>
-<xacro:rr_port_base_y_side name="x_base_front"  width="${x_axis_len}" len="${y_track_width}" height="${y_track_height}" weight="${y_bar_weight}" />
-<xacro:rr_port_base_y_side name="x_base_back"  width="${x_axis_len}" len="${y_track_width}" height="${y_track_height}" weight="${y_bar_weight}" />
+<xacro:rr_portal_bar name="x_base_front"  width="${x_axis_len}" len="${y_track_width}" height="${y_track_height}" weight="${x_base_bar_weight}" />
+<xacro:rr_portal_bar name="x_base_back"  width="${x_axis_len}" len="${y_track_width}" height="${y_track_height}" weight="${x_base_bar_weight}" />
 <joint name="joint_y_track_left_x_base_front" type="fixed">
 	<parent link="y_track_left" />

File: def/test_robots/portalbot/properties.xacro (robot description, xacro)
@@ -7,12 +7,14 @@
 <xacro:property name="x_track_width"  value="0.20" />
 <xacro:property name="x_track_height" value="0.05" />
+<xacro:property name="x_bar_weight" value="1.5" />
 <xacro:property name="y_track_width"  value="${x_track_height}" />
 <xacro:property name="y_track_height" value="${x_track_width}" />
 <xacro:property name="y_bar_weight" value="1.5" />
+<xacro:property name="x_base_bar_weight" value="1.5" />
 <xacro:property name="z_track_width"  value="${y_track_width}" />
 <xacro:property name="z_track_height" value="${x_track_height}" />
 <!-- Axis length in meters -->
-<xacro:property name="x_axis_len"  value="1.0" />
-<xacro:property name="y_axis_len"  value="2.0" />
-<xacro:property name="z_axis_len"  value="1.5" />
+<xacro:property name="x_axis_len"  value="$(arg x_axis_len)" />
+<xacro:property name="y_axis_len"  value="$(arg y_axis_len)" />
+<xacro:property name="z_axis_len"  value="$(arg z_axis_len)" />
 </robot>

Commit message: add portal frame

File: def/test_robots/portalbot.xacro (robot description, xacro)
@@ -8,3 +8,4 @@
 <xacro:include filename="$(find h4r_rapid_robot_xacros)/def/test_robots/portalbot/base.xacro"/>
 <xacro:include filename="$(find h4r_rapid_robot_xacros)/def/test_robots/portalbot/portal.xacro"/>
+<xacro:include filename="$(find h4r_rapid_robot_xacros)/def/test_robots/portalbot/x_axis.xacro"/>
 </robot>

File: def/test_robots/portalbot/base.xacro (robot description, xacro)
@@ -4,21 +4,4 @@
        xmlns:interface="http://playerstage.sourceforge.net/gazebo/xmlschema/#interface"
        xmlns:xacro="http://ros.org/wiki/xacro">
-<xacro:macro name="rr_port_base_y_side" params="name width len height weight">
-<link name="${name}">
-	<xacro:rr_inertia_box_solid x="${width}"
-		                        y="${len}"
-		                        z="${height}"
-		                        mass="${weight}">
-    <origin xyz="0 0 0" rpy="0 0 0" />
-    </xacro:rr_inertia_box_solid>
-	<visual>
-		<geometry><box size="${width} ${len} ${height}" /></geometry>
-		<material name="rr_m_gray_tp"/>
-	</visual>
-	<collision>
-		<geometry><box size="${width} ${len} ${height}" /></geometry>
-	</collision>
-</link>
-</xacro:macro>
 <xacro:rr_portal_bar name="y_track_left"  width="${y_track_width}" len="${y_axis_len}" height="${y_track_height}" weight="${y_bar_weight}" />
 <xacro:rr_portal_bar name="y_track_right" width="${y_track_width}" len="${y_axis_len}" height="${y_track_height}" weight="${y_bar_weight}" />

File: def/test_robots/portalbot/portal.xacro (robot description, xacro)
@@ -4,3 +4,17 @@
        xmlns:interface="http://playerstage.sourceforge.net/gazebo/xmlschema/#interface"
        xmlns:xacro="http://ros.org/wiki/xacro">
+	   <xacro:rr_portal_bar name="z_frame_left"  width="${z_frame_bar_width}" len="${z_frame_bar_height}" height="${z_frame_bar_length}" weight="${z_frame_bar_weight}" />
+       <xacro:rr_portal_bar name="z_frame_right" width="${z_frame_bar_width}" len="${z_frame_bar_height}" height="${z_frame_bar_length}" weight="${z_frame_bar_weight}" />
+       <joint name="joint_z_frame_left_z_frame_right" type="fixed">
+			<parent link="z_frame_left" />
+			<child  link="z_frame_right" />
+			<origin xyz="${x_axis_len+z_frame_bar_width} 0 0" rpy="0 0 0" />
+	   </joint>
+	  <joint name="joint_y_axis" type="prismatic">
+			<parent link="y_track_left" />
+			<child  link="z_frame_left" />
+			<origin xyz="0 0 ${z_axis_len/2 + y_track_height/2}" rpy="0 0 0" />
+		    <limit effort="1000.0" lower="-15" upper="15" velocity="30.0"/>
+      		<axis xyz="0 1 0"/>
+      </joint>
 </robot>

File: def/test_robots/portalbot/properties.xacro (robot description, xacro)
@@ -4,4 +4,8 @@
        xmlns:interface="http://playerstage.sourceforge.net/gazebo/xmlschema/#interface"
        xmlns:xacro="http://ros.org/wiki/xacro">
+<!-- Axis length in meters -->
+<xacro:property name="x_axis_len"  value="$(arg x_axis_len)" />
+<xacro:property name="y_axis_len"  value="$(arg y_axis_len)" />
+<xacro:property name="z_axis_len"  value="$(arg z_axis_len)" />
 <!-- Axis bar dimensions -->
 <xacro:property name="x_track_width"  value="0.20" />
@@ -12,9 +16,7 @@
 <xacro:property name="y_bar_weight" value="1.5" />
 <xacro:property name="x_base_bar_weight" value="1.5" />
-<xacro:property name="z_track_width"  value="${y_track_width}" />
-<xacro:property name="z_track_height" value="${x_track_height}" />
-<!-- Axis length in meters -->
-<xacro:property name="x_axis_len"  value="$(arg x_axis_len)" />
-<xacro:property name="y_axis_len"  value="$(arg y_axis_len)" />
-<xacro:property name="z_axis_len"  value="$(arg z_axis_len)" />
+<xacro:property name="z_frame_bar_width"  value="${y_track_width}" />
+<xacro:property name="z_frame_bar_height" value="${x_track_height}" />
+<xacro:property name="z_frame_bar_length" value="${z_axis_len-y_track_height+x_track_width}" />
+<xacro:property name="z_frame_bar_weight" value="1.5" />
 </robot>
