Commit message: first portal model, but needs changes...

File: def/material/materials.xacro (robot description, xacro)
@@ -20,3 +20,4 @@
 <xacro:rr_mat_color_def color="black" rgba="0 0 0 1" />
 <xacro:rr_mat_color_def color="gray_tp" rgba="0.5 0.5 0.5 .9" />
+<xacro:rr_mat_color_def color="gray" rgba="0.7 0.7 0.7 1" />
 </robot>

File: def/test_robots/portalbot/bar.xacro (robot description, xacro)
@@ -14,5 +14,5 @@
 	<visual>
 		<geometry><box size="${width} ${len} ${height}" /></geometry>
-		<material name="rr_m_gray_tp"/>
+		<material name="rr_m_gray"/>
 	</visual>
 	<collision>

File: def/test_robots/portalbot/properties.xacro (robot description, xacro)
@@ -12,4 +12,8 @@
 <xacro:property name="x_track_height" value="0.05" />
 <xacro:property name="x_bar_weight" value="1.5" />
+<xacro:property name="x_slider_width" value="0.2" />
+<xacro:property name="x_slider_height" value="0.2" />
+<xacro:property name="x_slider_len" value="0.05" />
+<xacro:property name="x_slider_weight" value="0.2" />
 <xacro:property name="y_track_width"  value="${x_track_height}" />
 <xacro:property name="y_track_height" value="${x_track_width}" />
@@ -20,3 +24,7 @@
 <xacro:property name="z_frame_bar_length" value="${z_axis_len-y_track_height+x_track_width}" />
 <xacro:property name="z_frame_bar_weight" value="1.5" />
+<xacro:property name="z_slider_len"  value="${z_axis_len+x_slider_height}" />
+<xacro:property name="z_slider_height" value="0.05" />
+<xacro:property name="z_slider_width" value="0.10" />
+<xacro:property name="z_frame_bar_weight" value="1.5" />
 </robot>

File: def/test_robots/portalbot/x_axis.xacro (robot description, xacro)
@@ -10,3 +10,11 @@
 		<origin xyz="${x_axis_len/2+z_frame_bar_width/2} 0 ${z_frame_bar_length/2-x_track_width/2}" rpy="0 0 0" />
    </joint>
+   	  <joint name="joint_x_axis" type="prismatic">
+			<parent link="x_track" />
+			<child  link="x_slider" />
+			<origin xyz="0 ${x_slider_len/2 + x_track_height/2} 0" rpy="0 0 0" />
+		    <limit effort="1000.0" lower="-15" upper="15" velocity="30.0"/>
+      		<axis xyz="1 0 0"/>
+      </joint>
+   <xacro:rr_portal_bar name="x_slider"  width="${x_slider_width}" len="${x_slider_len}" height="${x_slider_height}" weight="${x_slider_weight}" />
 </robot>
