Commit message: rename rr_portal_bar to rr_portal_element
also rename size params into (xyz)_size

File: def/test_robots/portalbot/bar.xacro (robot description, xacro)
@@ -4,18 +4,18 @@
        xmlns:interface="http://playerstage.sourceforge.net/gazebo/xmlschema/#interface"
        xmlns:xacro="http://ros.org/wiki/xacro">
-<xacro:macro name="rr_portal_bar" params="name width len height weight">
+<xacro:macro name="rr_portal_element" params="name x_size y_size z_size weight">
 <link name="${name}">
-	<xacro:rr_inertia_box_solid x="${width}"
-		                        y="${len}"
-		                        z="${height}"
+	<xacro:rr_inertia_box_solid x="${x_size}"
+		                        y="${y_size}"
+		                        z="${z_size}"
 		                        mass="${weight}">
     <origin xyz="0 0 0" rpy="0 0 0" />
     </xacro:rr_inertia_box_solid>
 	<visual>
-		<geometry><box size="${width} ${len} ${height}" /></geometry>
+		<geometry><box size="${x_size} ${y_size} ${z_size}" /></geometry>
 		<material name="rr_m_gray"/>
 	</visual>
 	<collision>
-		<geometry><box size="${width} ${len} ${height}" /></geometry>
+		<geometry><box size="${x_size} ${y_size} ${z_size}" /></geometry>
 	</collision>
 </link>

File: def/test_robots/portalbot/base.xacro (robot description, xacro)
@@ -4,6 +4,6 @@
        xmlns:interface="http://playerstage.sourceforge.net/gazebo/xmlschema/#interface"
        xmlns:xacro="http://ros.org/wiki/xacro">
-<xacro:rr_portal_bar name="y_track_left"  width="${y_track_width}" len="${y_axis_len}" height="${y_track_height}" weight="${y_bar_weight}" />
-<xacro:rr_portal_bar name="y_track_right" width="${y_track_width}" len="${y_axis_len}" height="${y_track_height}" weight="${y_bar_weight}" />
+<xacro:rr_portal_element name="y_track_left"  x_size="${y_track_width}" y_size="${y_axis_len}" z_size="${y_track_height}" weight="${y_bar_weight}" />
+<xacro:rr_portal_element name="y_track_right"  x_size="${y_track_width}" y_size="${y_axis_len}" z_size="${y_track_height}" weight="${y_bar_weight}" />
 <joint name="joint_y_track_right_left" type="fixed">
 	<parent link="y_track_left" />
@@ -11,6 +11,6 @@
 	<origin xyz="${x_axis_len + y_track_width} 0 0" rpy="0 0 0" />
 </joint>
-<xacro:rr_portal_bar name="x_base_front"  width="${x_axis_len}" len="${y_track_width}" height="${y_track_height}" weight="${x_base_bar_weight}" />
-<xacro:rr_portal_bar name="x_base_back"  width="${x_axis_len}" len="${y_track_width}" height="${y_track_height}" weight="${x_base_bar_weight}" />
+<xacro:rr_portal_element name="x_base_front"  x_size="${x_axis_len}" y_size="${y_track_width}" z_size="${y_track_height}" weight="${x_base_bar_weight}" />
+<xacro:rr_portal_element name="x_base_back"  x_size="${x_axis_len}" y_size="${y_track_width}" z_size="${y_track_height}" weight="${x_base_bar_weight}" />
 <joint name="joint_y_track_left_x_base_front" type="fixed">
 	<parent link="y_track_left" />

File: def/test_robots/portalbot/portal.xacro (robot description, xacro)
@@ -4,6 +4,6 @@
        xmlns:interface="http://playerstage.sourceforge.net/gazebo/xmlschema/#interface"
        xmlns:xacro="http://ros.org/wiki/xacro">
-	   <xacro:rr_portal_bar name="z_frame_left"  width="${z_frame_bar_width}" len="${z_frame_bar_height}" height="${z_frame_bar_length}" weight="${z_frame_bar_weight}" />
-       <xacro:rr_portal_bar name="z_frame_right" width="${z_frame_bar_width}" len="${z_frame_bar_height}" height="${z_frame_bar_length}" weight="${z_frame_bar_weight}" />
+	   <xacro:rr_portal_element name="z_frame_left"  x_size="${z_frame_bar_width}" y_size="${z_frame_bar_height}" z_size="${z_frame_bar_length}" weight="${z_frame_bar_weight}" />
+       <xacro:rr_portal_element name="z_frame_right"  x_size="${z_frame_bar_width}" y_size="${z_frame_bar_height}" z_size="${z_frame_bar_length}" weight="${z_frame_bar_weight}" />
        <joint name="joint_z_frame_left_z_frame_right" type="fixed">
 			<parent link="z_frame_left" />

File: def/test_robots/portalbot/x_axis.xacro (robot description, xacro)
@@ -4,5 +4,5 @@
 xmlns:interface="http://playerstage.sourceforge.net/gazebo/xmlschema/#interface"
 xmlns:xacro="http://ros.org/wiki/xacro">
-   <xacro:rr_portal_bar name="x_track"  width="${x_axis_len}" len="${x_track_height}" height="${x_track_width}" weight="${x_bar_weight}" />
+   <xacro:rr_portal_element name="x_track"  x_size="${x_axis_len}" y_size="${x_track_height}" z_size="${x_track_width}" weight="${x_bar_weight}" />
    <joint name="joint_z_frame_x_track" type="fixed">
 		<parent link="z_frame_left" />
@@ -17,4 +17,4 @@
       		<axis xyz="1 0 0"/>
       </joint>
-   <xacro:rr_portal_bar name="x_slider"  width="${x_slider_width}" len="${x_slider_len}" height="${x_slider_height}" weight="${x_slider_weight}" />
+   <xacro:rr_portal_element name="x_slider"  x_size="${x_slider_width}" y_size="${x_slider_len}" z_size="${x_slider_height}" weight="${x_slider_weight}" />
 </robot>

File: def/test_robots/portalbot/z_axis.xacro (robot description, xacro)
@@ -4,5 +4,5 @@
 xmlns:interface="http://playerstage.sourceforge.net/gazebo/xmlschema/#interface"
 xmlns:xacro="http://ros.org/wiki/xacro">
-   <xacro:rr_portal_bar name="z_slider"  width="${z_slider_width}" len="${z_slider_height}" height="${z_slider_len}" weight="${x_slider_weight}" />
+   <xacro:rr_portal_element name="z_slider"  x_size="${z_slider_width}" y_size="${z_slider_height}" z_size="${z_slider_len}" weight="${x_slider_weight}" />
     <joint name="joint_x_slider_z_axis" type="prismatic">
 			<parent link="x_slider" />
