Commit message: heavy refactoring, renaming rebuilding ->  portal -> gantry_bot

File: def/joints/linear_axis.xacro (robot description, xacro)
@@ -22,5 +22,5 @@
 			<child  link="${child}" />
 			<origin xyz="${origin_x} ${origin_y} ${origin_z}" rpy="${origin_R} ${origin_P} ${origin_Y}" />
-		    <limit effort="${effort}" lower="${velocity}" upper="${upper}" velocity="${velocity}"/>
+		    <limit effort="${effort}" lower="${lower}" upper="${upper}" velocity="${velocity}"/>
 			<xacro:if value="${axis == 'x'}">
 				<axis xyz="1 0 0"/>

File: def/test_robots/gantry_bot/element.xacro (robot description, xacro)
@@ -14,5 +14,5 @@
 	<visual>
 		<geometry><box size="${x_size} ${y_size} ${z_size}" /></geometry>
-		<material name="rr_m_gray"/>
+		<material name="rr_m_gray_tp"/>
 	</visual>
 	<collision>

Commit message: add ros_control interface to joints

File: def/joints/linear_axis.xacro (robot description, xacro)
@@ -17,4 +17,10 @@
 											  velocity
 											  axis
+											  ros_control:=false
+											  ros_control_actuator:='motor1'
+											  ros_control_effort:=false
+											  ros_control_velocity:=false
+											  ros_control_position:=false
+											  ros_control_reduction:=1
 											  ">
    	  <joint name="joint_linear_${parent}_${child}" type="prismatic">
@@ -33,4 +39,13 @@
 			</xacro:if>
       </joint>
+     <xacro:if value="${ros_control}">
+		<xacro:rr_roscontrol_simple_joint_transmission
+			joint="joint_linear_${parent}_${child}"
+			actuator="${ros_control_actuator}"
+			effort="${ros_control_effort}"
+			velocity="${ros_control_velocity}"
+			position="${ros_control_position}"
+		  	reduction="${ros_control_reduction}" />
+     </xacro:if>
 </xacro:macro>
 </robot>

File: def/rapid_robot.xacro (robot description, xacro)
@@ -26,4 +26,5 @@
 <xacro:include filename="$(find h4r_rapid_robot_xacros)/def/drive/diff_drive.xacro" />
 <!-- Joints -->
+<xacro:include filename="$(find h4r_rapid_robot_xacros)/def/joints/ros_control.xacro" />
 <xacro:include filename="$(find h4r_rapid_robot_xacros)/def/joints/fixed.xacro" />
 <xacro:include filename="$(find h4r_rapid_robot_xacros)/def/joints/linear_axis.xacro" />

File: def/test_robots/gantry_bot.xacro (robot description, xacro)
@@ -9,3 +9,5 @@
 <xacro:include filename="$(find h4r_rapid_robot_xacros)/def/test_robots/gantry_bot/boom.xacro"/>
 <xacro:include filename="$(find h4r_rapid_robot_xacros)/def/test_robots/gantry_bot/vertical.xacro"/>
+<xacro:include filename="$(find h4r_rapid_robot_xacros)/def/test_robots/gantry_bot/feet.xacro"/>
+<xacro:rr_roscontrol_controller />
 </robot>

File: def/test_robots/gantry_bot/boom.xacro (robot description, xacro)
@@ -30,4 +30,7 @@
 							 upper="15"
 							 velocity="30"
-							 axis="x"/>
+							 axis="y"
+	   						 ros_control="${ros_control}"
+	   						 ros_control_position="true"
+	   						/>
 </robot>

File: def/test_robots/gantry_bot/properties.xacro (robot description, xacro)
@@ -23,8 +23,8 @@
 <xacro:property name="boom_height"  		value="0.10" />
 <xacro:property name="boom_weight"  		value="1.0" />
-<xacro:property name="boom_slider_length"  		value="0.35" />
-<xacro:property name="boom_slider_width"   		value="0.05" />
-<xacro:property name="boom_slider_height"  		value="0.35" />
-<xacro:property name="boom_slider_weight"  		value="1.0" />
+<xacro:property name="boom_slider_length"  	value="0.35" />
+<xacro:property name="boom_slider_width"   	value="0.05" />
+<xacro:property name="boom_slider_height"  	value="0.35" />
+<xacro:property name="boom_slider_weight"  	value="1.0" />
 <xacro:property name="vertical_length"  	value="1.5" />
 <xacro:property name="vertical_width"   	value="0.20" />

File: def/test_robots/gantry_bot/rails.xacro (robot description, xacro)
@@ -30,4 +30,7 @@
 				      upper="${rail_length - rail_slider_width}"
 					  velocity="1"
-					  axis="x"/>
+					  axis="x"
+					  ros_control="${ros_control}"
+	   				  ros_control_position="true"
+						/>
 </robot>

File: def/test_robots/gantry_bot/vertical.xacro (robot description, xacro)
@@ -11,7 +11,10 @@
 					 origin_x="${-(vertical_height/2+boom_slider_width/2)}"
 					 effort="1000.0"
-					 lower ="-15"
-					 upper="15"
+					 lower ="0"
+					 upper="1"
 					 velocity="30"
-					 axis="z"/>
+					 axis="z"
+					 ros_control="${ros_control}"
+	   				 ros_control_position="true"
+					/>
 </robot>

Commit message: add ros_control config for gantry_bot

File: def/joints/linear_axis.xacro (robot description, xacro)
@@ -23,6 +23,13 @@
 											  ros_control_position:=false
 											  ros_control_reduction:=1
+											  joint_name=''
 											  ">
-   	  <joint name="joint_linear_${parent}_${child}" type="prismatic">
+	<xacro:if value="${joint_name == ''}">
+		 <xacro:property name="joint_name_in" value="joint_linear_${parent}_${child}" />
+	</xacro:if>
+	<xacro:unless value="${joint_name == ''}">
+		 <xacro:property name="joint_name_in" value="${joint_name}" />
+	</xacro:unless>
+   	  <joint name="${joint_name_in}" type="prismatic">
 			<parent link="${parent}" />
 			<child  link="${child}" />
@@ -41,5 +48,5 @@
      <xacro:if value="${ros_control}">
 		<xacro:rr_roscontrol_simple_joint_transmission
-			joint="joint_linear_${parent}_${child}"
+			joint="${joint_name_in}"
 			actuator="${ros_control_actuator}"
 			effort="${ros_control_effort}"

File: def/test_robots/gantry_bot.xacro (robot description, xacro)
@@ -6,4 +6,5 @@
 <xacro:include filename="$(find h4r_rapid_robot_xacros)/def/test_robots/gantry_bot/element.xacro"/>
 <xacro:include filename="$(find h4r_rapid_robot_xacros)/def/test_robots/gantry_bot/properties.xacro"/>
+<xacro:include filename="$(find h4r_rapid_robot_xacros)/def/test_robots/gantry_bot/base_link.xacro"/>
 <xacro:include filename="$(find h4r_rapid_robot_xacros)/def/test_robots/gantry_bot/rails.xacro"/>
 <xacro:include filename="$(find h4r_rapid_robot_xacros)/def/test_robots/gantry_bot/boom.xacro"/>

File: def/test_robots/gantry_bot/boom.xacro (robot description, xacro)
@@ -33,4 +33,5 @@
 	   						 ros_control="${ros_control}"
 	   						 ros_control_position="true"
-	   						/>
+	   						 joint_name="boom_joint"
+   						/>
 </robot>

File: def/test_robots/gantry_bot/rails.xacro (robot description, xacro)
@@ -33,4 +33,5 @@
 					  ros_control="${ros_control}"
 	   				  ros_control_position="true"
+					  joint_name="rail_joint"
 						/>
 </robot>

File: def/test_robots/gantry_bot/vertical.xacro (robot description, xacro)
@@ -17,4 +17,5 @@
 					 ros_control="${ros_control}"
 	   				 ros_control_position="true"
+					 joint_name="vertical_joint"
 					/>
 </robot>
