Commit message: disable world macro needs fixing

File: def/rapid_robot.xacro (robot description, xacro)
@@ -35,3 +35,8 @@
 <!-- Video -->
 <xacro:include filename="$(find h4r_rapid_robot_xacros)/def/video/screen.xacro"/>
+<!-- World 	-->
+<xacro:include filename="$(find h4r_rapid_robot_xacros)/def/world/static.xacro"/>
+<!--
+<xacro:include filename="$(find h4r_rapid_robot_xacros)/def/world/world_joint.xacro"/>
+-->
 </robot>

File: def/world/world_joint.xacro (robot description, xacro)
@@ -6,9 +6,9 @@
 <xacro:macro name="rr_world_joint" params="root_link:='base_link' default:=true" />
 <xacro:arg name="world_joint" default="${default}"/>
-<xacro:if value="$(arg world_joint)">
+<xacro:if value="$(arg root_link)">
   <link name="world"/>
   <joint name="fixed" type="fixed">
     <parent link="world"/>
-    <child link="${base_link}"/>
+    <child link="$(arg root_link)"/>
   </joint>
 </xacro:if>
