Commit message: fixing multiple axis

File: def/test_robots/gantry_bot/base_link.xacro (robot description, xacro)
@@ -5,4 +5,4 @@
        xmlns:xacro="http://ros.org/wiki/xacro">
        <link name="base_link" />
-       <xacro:rr_joint_fixed parent="base_link" child="rail_left" origin_x="${rail_length/2}" origin_y="${-rail_width/2}" />
+       <xacro:rr_joint_fixed parent="base_link" child="rail_left" origin_x="${rail_length/2}" origin_y="${-rail_width/2}" origin_z="${(foot_length+rail_height/2)}" />
 </robot>

File: def/test_robots/gantry_bot/boom.xacro (robot description, xacro)
@@ -18,5 +18,5 @@
 <xacro:rr_portal_element name="boom" x_size="${boom_width}" y_size="${boom_length}" z_size="${boom_height}" weight="${boom_weight}" />
 <xacro:rr_joint_fixed parent="boom_support_left" child="boom"
-					  origin_x="${boom_support_length/2-boom_width/2}"
+					  origin_x="${-(boom_support_length/2-boom_width/2)}"
 					  origin_y="${boom_length/2-boom_support_width/2}"
    					  origin_z="${boom_support_height/2+boom_height/2}"/>
@@ -26,7 +26,8 @@
 	                         child="boom_slider"
 	   						 origin_x="${-(boom_slider_width/2+boom_width/2)}"
+							 origin_y="${(boom_length-boom_slider_length)/2}"
 	   						 effort="1000.0"
-							 lower ="-15"
-							 upper="15"
+							 lower ="0"
+							 upper="${boom_length-boom_slider_length}"
 							 velocity="30"
 							 axis="y"

File: def/test_robots/gantry_bot/properties.xacro (robot description, xacro)
@@ -17,4 +17,6 @@
 <xacro:property name="vertical_length"  	value="$(arg vertical_len)" />
 <xacro:property name="boom_support_height"  value="$(arg boom_support_height)" />
+<xacro:property name="vertical_offset"  	value="$(arg vertical_offset)" />
+<xacro:property name="vertical_axis_slider_offset"  value="$(arg vertical_axis_slider_offset)" />
 <xacro:property name="rail_width"   		value="${vslot2040_width}" />
 <xacro:property name="rail_height"  		value="${vslot2040_height}" />
@@ -41,5 +43,4 @@
 <xacro:property name="vertical_height"  	value="${vslot2020_width}" />
 <xacro:property name="vertical_weight"  	value="${vertical_length*vslot2020_weight_per_meter}" />
-<xacro:property name="vertical_axis_slider_offset"  value="0.05" />
 <xacro:property name="foot_length"  	value="0.1" />
 <xacro:property name="foot_width"   	value="0.05" />

File: def/test_robots/gantry_bot/vertical.xacro (robot description, xacro)
@@ -11,7 +11,8 @@
 					 origin_x="${-(vertical_height/2+boom_slider_width/2)}"
  					 origin_y="${vertical_axis_slider_offset}"
+					 origin_z="${vertical_length/2-vertical_offset}"
 					 effort="1000.0"
 					 lower ="0"
-					 upper="1"
+					 upper="${vertical_length}"
 					 velocity="30"
 					 axis="z"
