Commit message: add end offset settings for endstops (not working WTF?)

File: def/test_robots/gantry_bot/boom.xacro (robot description, xacro)
@@ -26,8 +26,8 @@
 	                         child="boom_slider"
 	   						 origin_x="${-(boom_slider_width/2+boom_width/2)}"
-							 origin_y="${(boom_length-boom_slider_length)/2}"
+							 origin_y="${(boom_length-boom_slider_length)/2-boom_length_offset_start}"
 	   						 effort="1000.0"
 							 lower ="0"
-							 upper="${boom_length-boom_slider_length}"
+							 upper="${boom_length-boom_slider_length-boom_length_offset_start-boom_length_offset_end}"
 							 velocity="30"
 							 axis="y"

File: def/test_robots/gantry_bot/properties.xacro (robot description, xacro)
@@ -14,8 +14,13 @@
 <xacro:property name="vslot2060_width"   		value="0.02" />
 <xacro:property name="rail_length"  		value="$(arg rail_len)" />
+<xacro:property name="rail_length_offset_start"  		value="$(arg rail_length_offset_start)" />
+<xacro:property name="rail_length_offset_end"  			value="$(arg rail_length_offset_end)" />
 <xacro:property name="boom_length"  		value="$(arg boom_len)" />
+<xacro:property name="boom_length_offset_start"  		value="$(arg boom_length_offset_start)" />
+<xacro:property name="boom_length_offset_end"  			value="$(arg boom_length_offset_end)" />
+<xacro:property name="boom_support_height"  value="$(arg boom_support_height)" />
 <xacro:property name="vertical_length"  	value="$(arg vertical_len)" />
-<xacro:property name="boom_support_height"  value="$(arg boom_support_height)" />
-<xacro:property name="vertical_offset"  	value="$(arg vertical_offset)" />
+<xacro:property name="vertical_length_offset_start"  	value="$(arg vertical_length_offset_start)" />
+<xacro:property name="vertical_length_offset_end"  		value="$(arg vertical_length_offset_end)" />
 <xacro:property name="vertical_axis_slider_offset"  value="$(arg vertical_axis_slider_offset)" />
 <xacro:property name="rail_width"   		value="${vslot2040_width}" />

File: def/test_robots/gantry_bot/rails.xacro (robot description, xacro)
@@ -24,9 +24,9 @@
 <xacro:rr_linear_axis parent="rail_left"
 	                  child="rail_slider_left"
-	   	              origin_x="${ -( (rail_length/2) - (rail_slider_length/2) )}"
+	   	              origin_x="${ -( (rail_length/2) - (rail_slider_length/2) ) + rail_length_offset_start}"
 					  origin_y="${ -( (rail_width/2)  + (rail_slider_width/2) )}"
 	   				  effort="1000.0"
 				      lower ="0"
-				      upper="${rail_length - rail_slider_width}"
+				      upper="${rail_length - rail_slider_width - rail_length_offset_start - rail_length_offset_end}"
 					  velocity="1"
 					  axis="x"

File: def/test_robots/gantry_bot/vertical.xacro (robot description, xacro)
@@ -11,8 +11,8 @@
 					 origin_x="${-(vertical_height/2+boom_slider_width/2)}"
  					 origin_y="${vertical_axis_slider_offset}"
-					 origin_z="${vertical_length/2-vertical_offset}"
+					 origin_z="${vertical_length/2-vertical_length_offset_start}"
 					 effort="1000.0"
 					 lower ="0"
-					 upper="${vertical_length}"
+					 upper="${vertical_length-vertical_length_offset_start-vertical_length_offset_end}"
 					 velocity="30"
 					 axis="z"
