Commit message: add density automatic weight calculation to simple box

File: def/simple/simple_box.xacro (robot description, xacro)
@@ -6,5 +6,6 @@
 >
 <xacro:macro name="rr_simple_box"
-	params="name x_size y_size z_size weight
+	params="name x_size y_size z_size
+	        weight:=1
             fric_mu1=100
             fric_mu2:=50
@@ -14,11 +15,18 @@
 	        gazebo_material:='Gazebo/White'
 	        rviz_material:='rr_m_gray_tp'
+			density:=0
 			"
 			>
 <link name="${name}">
+	<xacro:if value="${density==0}" >
+		<xacro:property name="mass" value="${weight}" />
+	</xacro:if>
+	<xacro:unless value="${density==0}" >
+		<xacro:property name="mass" value="${x_size*y_size*z_size*density}" />
+	</xacro:unless>
 	<xacro:rr_inertia_box_solid x="${x_size}"
 		                        y="${y_size}"
 		                        z="${z_size}"
-		                        mass="${weight}">
+		                        mass="${mass}">
     <origin xyz="0 0 0" rpy="0 0 0" />
     </xacro:rr_inertia_box_solid>
